File: OrangePie/5v buck.kicad_sch (KiCad schematic)
At the start: 0 parts

Commit message: Update rest of schematic
Parts:
- added C24, C26: 100nF 50V Y5V, Capacitor_SMD:C_0402_1005Metric, symbol Device:C_Small
- added C25: 10uF 50v, Capacitor_SMD:C_0805_2012Metric, symbol Device:C
- added C27, C28, C29, C30: 10uF, PCM_JLCPCB:C_1206, symbol PCM_JLCPCB-Capacitors:1206,10uF
- added C31, C32: 1uF 25V, Capacitor_SMD:C_0402_1005Metric, symbol Device:C_Small
- added C41: 47uF, Capacitor_SMD:CP_Elec_6.3x5.4, symbol Device:C_Polarized
- added L1: 6.8uH 12.5x12.5mm, Inductor_SMD:L_AVX_LMLP07A7, symbol Device:L
- added R14: 39k 1%, Resistor_SMD:R_0402_1005Metric, symbol Device:R
- added R15: 31.6k 1%, Resistor_SMD:R_0402_1005Metric, symbol Device:R
- added R16, R17: 10k 1%, Resistor_SMD:R_0402_1005Metric, symbol Device:R
- added U6: ~, Package_SO:Diodes_SO-8EP, symbol SY8205:SY8205
Connections:
- new net: R15.2, R17.1, U6.5 (FB)
- new net: C24.1, U6.1 (BST)
- new net: C24.2, L1.1, U6.2 (Lx)
- new net: R14.2, R16.1, U6.3 (EN)
- new net: C32.2, U6.4 (SS)
- new net: C31.2, U6.6 (VCC)
- new net 5V_OUT: C27.1, C28.1, C29.1, C30.1, L1.2, R15.1
- new net GND: C25.2, C26.2, C27.2, C28.2, C29.2, C30.2, C31.1, C32.1, C41.2, R16.2, R17.2, U6.9 (EPAD)
- new net Vin: C25.1, C26.1, C41.1, R14.1, U6.7 (Vin), U6.8 (Vin)
Other:
- note added: "1.2v tresh"
- note added: "6v UVLO"

Commit message: Add CH340 debug
Other:
- company: (none) -> ModuCard System
Changed lines of the file:
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@@
 	(generator_version "8.0")
 	(paper "A4")
+	(title_block
+		(date "2025-02-10")
+		(rev "A")
+		(company "ModuCard System")
+	)
 	(junction
 		(at 58.42 83.82)
