File: OrangePie/Audio Codec.kicad_sch (KiCad schematic)
At the start: 25 parts, among them J1 JST XH, U1 PCM2704CDBR, U2 TDA7052A, X1 X322512MSB4SI

Commit message: Add CH340 debug
Other:
- company: Artem Horiunov -> ModuCard System
Changed lines of the file:
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@@
 	(title_block
 		(title "PCM2704 USB SOUND OUTPUT")
-		(date "2025-02-08")
+		(date "2025-02-10")
 		(rev "A")
-		(company "Artem Horiunov")
+		(company "ModuCard System")
 		(comment 1 "DESIGNED IN POLAND")
 	)
