File: OrangePie/FAN controller.kicad_sch (KiCad schematic)
At the start: 9 parts, among them M1 Fan, Q1 AO3400A

Commit message: Add CH340 debug
Other:
- company: (none) -> ModuCard System
Changed lines of the file:
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@@
 	(generator_version "8.0")
 	(paper "A4")
+	(title_block
+		(date "2025-02-10")
+		(rev "A")
+		(company "ModuCard System")
+	)
 	(junction
 		(at 152.4 115.57)
