File: OrangePie/Power Oring.kicad_sch (KiCad schematic)
At the start: 0 parts

Commit message: Update rest of schematic
Parts:
- added C33, C34: 100nF 50V Y5V, Capacitor_SMD:C_0402_1005Metric, symbol Device:C_Small
- added Q2, Q3: AO3400, Package_TO_SOT_SMD:SOT-23, symbol Simulation_SPICE:NMOS
- added Q4: MMBT3904, PCM_JLCPCB:Q_SOT-23, symbol PCM_JLCPCB-Transistors:NPN,MMBT3904
- added R18, R22: 10kΩ, PCM_JLCPCB:R_0402, symbol PCM_JLCPCB-Resistors:0402,10kΩ
- added U7, U8: LM74700, Package_TO_SOT_SMD:SOT-23-6, symbol Power_Management:LM74700
Connections:
- new net: C33.2, U7.1 (VCAP)
- new net: C34.2, U8.1 (VCAP)
- new net: R22.2, U8.3 (EN)
- new net: Q3.1 (G), U8.5 (GATE)
- new net: Q4.3 (C), R18.2, U7.3 (EN)
- new net: Q2.1 (G), U7.5 (GATE)
- new net +5V: Q2.2 (D), Q3.2 (D), U7.4 (CATHODE), U8.4 (CATHODE)
- new net BUCK_IN: C33.1, Q2.3 (S), R18.1, U7.6 (ANODE)
- new net GND: Q4.2 (E), U7.2 (GND), U8.2 (GND)
- new net STDBY_IN: C34.1, Q3.3 (S), R22.1, U8.6 (ANODE)
- new net ~{STDBY EN}: Q4.1 (B)

Commit message: Add CH340 debug
Other:
- company: (none) -> ModuCard System
Changed lines of the file:
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@@
 	(generator_version "8.0")
 	(paper "A4")
+	(title_block
+		(date "2025-02-10")
+		(rev "A")
+		(company "ModuCard System")
+	)
 	(junction
 		(at 116.84 116.84)
