File: PCB source/Audio Codec.kicad_sch (KiCad schematic)
At the start: 25 parts, among them J1 JST XH, U1 PCM2704CDBR, U2 TDA7052A, X1 X322512MSB4SI

Commit message: Do Cleanup
Parts:
- renumbered C6 to C32, C3 to C33, C15 to C34, C14 to C35, C4 to C36, C5 to C37, C13 to C38, C12 to C39, C11 to C40, C1 to C41, C2 to C42, C10 to C43, C9 to C44, J1 to J3, R1 to R16, R2 to R17, R3 to R18, R5 to R19, R6 to R20, R7 to R21, R4 to R22, U2 to U8, U1 to U9
Connections:
- net +5V: now also U9.10 (VBUS); no longer R19.1, R22.2, U9.21 (HOST), U9.25 (TEST1), U9.26 (TEST0), U9.27 (~{SSPND}), U9.4 (PSEL), U9.7 (VDD)
- net VDD_{int}: now reaches C34.1
- net VDD_{int}: now also R19.1, R22.2, U9.21 (HOST), U9.25 (TEST1), U9.26 (TEST0), U9.27 (~{SSPND}), U9.4 (PSEL), U9.7 (VDD); no longer U9.10 (VBUS)
Other:
- moved on the sheet: C32, C33, C34, C35, C38, C39, C41
