File: PCB source/OrangePie.kicad_pcb (KiCad board)
At the start: 2 copper layers, 38 x 38 mm, 99 parts, among them J1 JST XH, J2 Orange pi 5 pro, J3 09031967921, M1 Fan, Q1 AO3400A, Q2 AO3400, Q3 AO3400, Q4 MMBT3904, U10 IP4234CZ6,115, U3 CH334R, U4 TJA1044GTK_3Z, U5 TJA1044GTK_3Z, U7 LM74700, U8 LM74700, U9 STM32G431C8Tx, X1 X322512MSB4SI, Y1 12MHz

Commit message: Do Cleanup
Parts:
- removed U8: LM74700, Package_TO_SOT_SMD:SOT-23-6
- removed U9: STM32G431C8Tx, Package_QFP:LQFP-48_7x7mm_P0.5mm
- added BTN1: TL2243, TL2243:TL2243, F.Cu at (137.6, 45.8)
- added C50: 47uF, Capacitor_SMD:CP_Elec_6.3x5.4, F.Cu at (188.2, 87.6)
- added C51: 100nF, PCM_JLCPCB:C_0402, F.Cu at (191.8, 112.1)
- added C52: 100nF, PCM_JLCPCB:C_0402, F.Cu at (191.8, 114.0)
- added C53: 20pF, Capacitor_SMD:C_0402_1005Metric, F.Cu at (191.8, 108.3)
- added C54: 20pF, Capacitor_SMD:C_0402_1005Metric, F.Cu at (191.8, 110.2)
- added C55: 100nF, PCM_JLCPCB:C_0402, F.Cu at (178.3, 63.7)
- added C56: 10uF, PCM_JLCPCB:C_0805, F.Cu at (179.1, 80.0)
- added D4: 1N4002W, PCM_JLCPCB:D_SOD-123FL, F.Cu at (201.3, 72.6)
- added J4: Connector, USB-TYPE-C-16P, USB_C_Upright16pin:MOLEX_2169890001, F.Cu at (169.1, 57.7)
- added LED1: FixLed307, FixLed307:FixLed307, F.Cu at (145.4, 45.1)
- added R23: 0Ω, PCM_JLCPCB:R_0402, F.Cu at (178.3, 65.5)
- added R24: 0Ω, PCM_JLCPCB:R_0402, F.Cu at (178.3, 67.4)
- added R25: 1.5kΩ, PCM_JLCPCB:R_0402, F.Cu at (178.3, 69.2)
- added R26: 10kΩ, PCM_JLCPCB:R_0402, F.Cu at (178.3, 71.1)
- added R27: 5.1kΩ, PCM_JLCPCB:R_0402, F.Cu at (178.3, 72.9)
- added R28: 5.1kΩ, PCM_JLCPCB:R_0402, F.Cu at (212.8, 58.1)
- added R29: 22Ω, PCM_JLCPCB:R_0402, F.Cu at (212.8, 60.0)
- added R30: 22Ω, PCM_JLCPCB:R_0402, F.Cu at (212.8, 61.8)
- added R31: 1kΩ, PCM_JLCPCB:R_0402, F.Cu at (212.8, 63.7)
- added U1: IP4234CZ6,115, Package_TO_SOT_SMD:SC-74-6_1.55x2.9mm_P0.95mm, F.Cu at (156.0, 113.1)
- added U11: CH340G, Package_SO:SOIC-16_3.9x9.9mm_P1.27mm, F.Cu at (186.2, 108.7)
- added U12: IP4234CZ6, Package_TO_SOT_SMD:SC-74-6_1.55x2.9mm_P0.95mm, F.Cu at (179.6, 76.3)
- added U2: ~, Package_SO:Diodes_SO-8EP, F.Cu at (154.3, 90.6)
- added Y2: 12MHz C7424717, Crystal:Crystal_SMD_3225-4Pin_3.2x2.5mm, F.Cu at (193.0, 105.1)
- C10: value 22pF -> 100nF 50V Y5V; footprint PCM_JLCPCB:C_0402 -> Capacitor_SMD:C_0402_1005Metric
- C11: value 47uF -> 10uF; footprint Capacitor_SMD:CP_Elec_6.3x5.4 -> PCM_JLCPCB:C_1206
- C12, C13, C14: value 1uF -> 10uF; footprint PCM_JLCPCB:C_0402 -> PCM_JLCPCB:C_1206
- C15: value 1uF -> 100nF 50V Y5V; footprint PCM_JLCPCB:C_0402 -> Capacitor_SMD:C_0402_1005Metric
- C16: value 10uF -> 1uF
- C17: value 100nF -> 1uF
- C18, C19, C20, C21: footprint Capacitor_SMD:C_0402_1005Metric -> PCM_JLCPCB:C_0402
- C2: value 1uF -> 47uF; footprint PCM_JLCPCB:C_0402 -> Capacitor_SMD:CP_Elec_6.3x5.4
- C22, C23: value 47uF -> 100nF; footprint Capacitor_SMD:CP_Elec_6.3x5.4 -> PCM_JLCPCB:C_0402
- C24: value 100nF 50V Y5V -> 10uF; footprint Capacitor_SMD:C_0402_1005Metric -> PCM_JLCPCB:C_0402
- C25: value 10uF 50v -> 100n; footprint Capacitor_SMD:C_0805_2012Metric -> Capacitor_SMD:C_0402_1005Metric
- C27: value 10uF -> 100nF 50V Y5V; footprint PCM_JLCPCB:C_1206 -> Capacitor_SMD:C_0402_1005Metric
- C28, C29, C30, C36: value 10uF -> 100nF; footprint PCM_JLCPCB:C_1206 -> PCM_JLCPCB:C_0402
- C3, C5: footprint PCM_JLCPCB:C_0805 -> PCM_JLCPCB:C_1206
- C31, C32: value 1uF 25V -> 100nF; footprint Capacitor_SMD:C_0402_1005Metric -> PCM_JLCPCB:C_0402
- C33: value 100nF 50V Y5V -> 10uF; footprint Capacitor_SMD:C_0402_1005Metric -> PCM_JLCPCB:C_0805
- C34: value 100nF 50V Y5V -> 1uF; footprint Capacitor_SMD:C_0402_1005Metric -> PCM_JLCPCB:C_0402
- C35: value 47uF -> 1uF; footprint Capacitor_SMD:CP_Elec_6.3x5.4 -> PCM_JLCPCB:C_0402
- C37: footprint PCM_JLCPCB:C_1206 -> PCM_JLCPCB:C_0805
- C38, C39: value 10uF -> 1uF; footprint PCM_JLCPCB:C_1206 -> PCM_JLCPCB:C_0402
- C4, C6: value 100nF -> 10uF; footprint PCM_JLCPCB:C_0402 -> PCM_JLCPCB:C_1206
- C40: value 10uF -> 47uF; footprint PCM_JLCPCB:C_1206 -> Capacitor_SMD:CP_Elec_6.3x5.4
- C42: value 100n -> 1uF; footprint Capacitor_SMD:C_0402_1005Metric -> PCM_JLCPCB:C_0402
- C43, C44: value 100n -> 22pF; footprint Capacitor_SMD:C_0402_1005Metric -> PCM_JLCPCB:C_0402
- C45: value 100n -> 10uF; footprint Capacitor_SMD:C_0402_1005Metric -> PCM_JLCPCB:C_0402
- C46: value 1u -> 1uF; footprint Capacitor_SMD:C_0603_1608Metric -> PCM_JLCPCB:C_0402
- C47: value 4.7u -> 10uF; footprint Capacitor_SMD:C_0603_1608Metric -> PCM_JLCPCB:C_0402
- C48: value 10u -> 100nF; footprint Capacitor_SMD:C_0805_2012Metric -> PCM_JLCPCB:C_0402
- C49: value 100n -> 10uF; footprint Capacitor_SMD:C_0402_1005Metric -> PCM_JLCPCB:C_1206
- C7: value 1uF -> 100nF
- C8: value 10uF -> 47uF; footprint PCM_JLCPCB:C_0402 -> Capacitor_SMD:CP_Elec_6.3x5.4
- C9: value 22pF -> 10uF 50v; footprint PCM_JLCPCB:C_0402 -> Capacitor_SMD:C_0805_2012Metric
- D1: value 1N4002W -> Green; footprint PCM_JLCPCB:D_SOD-123FL -> PCM_JLCPCB:D_0603
- D2: value WORD_LED -> Green; footprint Diode_SMD:D_0603_1608Metric -> PCM_JLCPCB:D_0603
- D3: value STAT_LED -> Green; footprint Diode_SMD:D_0603_1608Metric -> PCM_JLCPCB:D_0603
- J1: value JST XH -> 09031967921; footprint Connector_JST:JST_XH_B2B-XH-AM_1x02_P2.50mm_Vertical -> Connector_DIN:DIN41612_R_3x32_Female_Horizontal_THT
- J3: value 09031967921 -> JST XH; footprint Connector_DIN:DIN41612_R_3x32_Female_Horizontal_THT -> Connector_JST:JST_XH_B2B-XH-AM_1x02_P2.50mm_Vertical
- Q1: value AO3400A -> AO3400
- Q2: value AO3400 -> MMBT3904; footprint Package_TO_SOT_SMD:SOT-23 -> PCM_JLCPCB:Q_SOT-23
- Q4: value MMBT3904 -> AO3400A; footprint PCM_JLCPCB:Q_SOT-23 -> Package_TO_SOT_SMD:SOT-23
- R1: value 220Ω -> 39k 1%; footprint PCM_JLCPCB:R_0402 -> Resistor_SMD:R_0402_1005Metric
- R10, R11: value 0Ω -> 1k; footprint PCM_JLCPCB:R_0402 -> Resistor_SMD:R_0402_1005Metric
- R13: value 1.5kΩ -> 10kΩ
- R14: value 39k 1% -> 10kΩ; footprint Resistor_SMD:R_0402_1005Metric -> PCM_JLCPCB:R_0402
- R15: value 31.6k 1% -> 10kΩ; footprint Resistor_SMD:R_0402_1005Metric -> PCM_JLCPCB:R_0402
- R16, R17: value 10k 1% -> 220Ω; footprint Resistor_SMD:R_0402_1005Metric -> PCM_JLCPCB:R_0402
- R19: value 10k -> 1.5kΩ; footprint Resistor_SMD:R_0402_1005Metric -> PCM_JLCPCB:R_0402
- R2: value 220Ω -> 31.6k 1%; footprint PCM_JLCPCB:R_0402 -> Resistor_SMD:R_0402_1005Metric
- R20, R21: value 1k -> 22Ω; footprint Resistor_SMD:R_0402_1005Metric -> PCM_JLCPCB:R_0402
- R22: value 10kΩ -> 1.5kΩ
- R3: value 10kΩ -> 10k 1%; footprint PCM_JLCPCB:R_0402 -> Resistor_SMD:R_0402_1005Metric
- R4: value 1.5kΩ -> 10k 1%; footprint PCM_JLCPCB:R_0402 -> Resistor_SMD:R_0402_1005Metric
- R5: value 1.5kΩ -> 10k; footprint PCM_JLCPCB:R_0402 -> Resistor_SMD:R_0402_1005Metric
- R6, R7: value 22Ω -> 1k; footprint PCM_JLCPCB:R_0402 -> Resistor_SMD:R_0402_1005Metric
- R8: value 10k -> 10kΩ; footprint Resistor_SMD:R_0402_1005Metric -> PCM_JLCPCB:R_0402
- TP1, TP2, TP3, TP4, TP5: footprint TestPoint:TestPoint_Pad_1.0x1.0mm -> TestPoint:TestPoint_Pad_D1.0mm
- U10: value IP4234CZ6,115 -> CH334R; footprint Package_TO_SOT_SMD:SC-74-6_1.55x2.9mm_P0.95mm -> Package_SO:QSOP-16_3.9x4.9mm_P0.635mm
- U3: value CH334R -> STM32G431C8Tx; footprint Package_SO:QSOP-16_3.9x4.9mm_P0.635mm -> Package_QFP:LQFP-48_7x7mm_P0.5mm
- U4, U5: value TJA1044GTK_3Z -> LM74700; footprint Package_SON:HVSON-8-1EP_3x3mm_P0.65mm_EP1.6x2.4mm -> Package_TO_SOT_SMD:SOT-23-6
- U6: value ~ -> TJA1044GTK_3Z; footprint Package_SO:Diodes_SO-8EP -> Package_SON:HVSON-8-1EP_3x3mm_P0.65mm_EP1.6x2.4mm
- U7: value LM74700 -> TJA1044GTK_3Z; footprint Package_TO_SOT_SMD:SOT-23-6 -> Package_SON:HVSON-8-1EP_3x3mm_P0.65mm_EP1.6x2.4mm
- moved R9 98.9 mm to (193.5, 74.8), turned to 0 degrees
- moved R8 96.9 mm to (193.5, 72.9), turned to 0 degrees
- moved U5 95.7 mm to (191.8, 69.8), turned to 0 degrees
- moved U4 94.5 mm to (191.8, 65.2), turned to 0 degrees
- moved D3 88.9 mm to (196.3, 88.5), turned to 0 degrees
- moved R21 86.0 mm to (193.8, 96.3), turned to 0 degrees
- moved C49 85.6 mm to (196.4, 85.2), turned to 0 degrees
- moved R20 84.2 mm to (193.8, 94.4), turned to 0 degrees
- moved R19 82.4 mm to (193.8, 92.6), turned to 0 degrees
- moved C21 71.0 mm to (168.1, 90.0), turned to 0 degrees
- moved U3 70.1 mm to (175.2, 89.2), turned to 0 degrees
- moved C19 70.0 mm to (168.1, 86.3), turned to 0 degrees
- moved C20 69.5 mm to (168.1, 88.1), turned to 0 degrees
- moved C17 69.0 mm to (158.7, 99.9), turned to 0 degrees
- moved C18 68.5 mm to (168.1, 84.4), turned to 0 degrees
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Connections:
- C1 pad 1: /Audio Codec/VCOM -> +5V
- C10 pad 1: Net-(U1-XTI) -> /DIN41612 connector/12v
- C11 pad 1: Net-(C11-Pad1) -> /5v buck/5V_OUT
- C11 pad 2: Net-(U2-+) -> GND
- C12 pad 1: Net-(U1-VCCP) -> /5v buck/5V_OUT
- C13 pad 1: Net-(U1-VCCR) -> /5v buck/5V_OUT
- C14 pad 1: Net-(U1-VCCL) -> /5v buck/5V_OUT
- C15 pad 1: Net-(U1-VBUS) -> /5v buck/5V_OUT
- C16 pad 1: +5V -> Net-(U2-VCC)
- C17 pad 1: +5V -> Net-(U2-SS)
- C18 pad 1: GND -> +3V3
- C18 pad 2: +5V -> GND
- C19 pad 1: GND -> +3V3
- C19 pad 2: +3V3 -> GND
- C2 pad 1: Net-(U2-V) -> +5V
- C20 pad 1: GND -> +3V3
- C20 pad 2: +5V -> GND
- C21 pad 1: GND -> +3V3
- C21 pad 2: +3V3 -> GND
- C22 pad 1: Net-(M1-+) -> +3V3
- C23 pad 1: +5V -> +3V3
- C24 pad 1: Net-(U6-BST) -> +3V3
- C24 pad 2: Net-(U6-Lx) -> GND
- C25 pad 1: /DIN41612 connector/12v -> /USB-CAN/NRST1
- C26 pad 1: /DIN41612 connector/12v -> /Power Oring/BUCK_IN
- C26 pad 2: GND -> Net-(U4-VCAP)
- C27 pad 1: /5v buck/5V_OUT -> /DIN41612 connector/5v_STDBY
- C27 pad 2: GND -> Net-(U5-VCAP)
- C28 pad 1: /5v buck/5V_OUT -> GND
- C28 pad 2: GND -> +5V
- C29 pad 1: /5v buck/5V_OUT -> +3V3
- C3 pad 1: GND -> +5V
- C3 pad 2: +5V -> GND
- C30 pad 1: /5v buck/5V_OUT -> GND
- C30 pad 2: GND -> +5V
- C31 pad 1: GND -> +3V3
- C31 pad 2: Net-(U6-VCC) -> GND
- C32 pad 1: GND -> +5V
- C32 pad 2: Net-(U6-SS) -> GND
- C33 pad 1: /5v buck/5V_OUT -> GND
- C33 pad 2: Net-(U7-VCAP) -> +5V
- C34 pad 1: /DIN41612 connector/5v_STDBY -> Net-(U9-VBUS)
- C34 pad 2: Net-(U8-VCAP) -> GND
- C35 pad 1: +5V -> Net-(U9-VCCL)
- C37 pad 1: +5V -> GND
- C37 pad 2: GND -> +5V
- C38 pad 1: +5V -> Net-(U9-VCCR)
- C39 pad 1: +5V -> Net-(U9-VCCP)
- C40 pad 1: Net-(M1-+) -> Net-(C40-Pad1)
- C40 pad 2: GND -> Net-(U8-+)
- C41 pad 1: /DIN41612 connector/12v -> /Audio Codec/VCOM
- C42 pad 1: +3V3 -> Net-(U8-V)
- C43 pad 1: +3V3 -> Net-(U9-XTI)
- C44 pad 1: +3V3 -> Net-(U9-XTO)
- C45 pad 1: +3V3 -> Net-(U10-VDD33)
- C46 pad 1: +3V3 -> Net-(U10-VDD33)
- C47 pad 1: +3V3 -> +5V
- C48 pad 1: +3V3 -> +5V
- C49 pad 1: /USB-CAN/NRST1 -> Net-(M1-+)
- C5 pad 1: GND -> +5V
- C5 pad 2: +5V -> GND
- C7 pad 1: Net-(U3-VDD33) -> Net-(U2-BST)
- C7 pad 2: GND -> Net-(U2-Lx)
- C8 pad 1: Net-(U3-VDD33) -> /DIN41612 connector/12v
- C9 pad 1: Net-(U1-XTO) -> /DIN41612 connector/12v
- D1 pad 1: Net-(M1-+) -> Net-(D1-Pad1)
- D1 pad 2: Net-(M1--) -> +3V3
- D2 pad 1: Net-(D2-K) -> Net-(D2-Pad1)
- D3 pad 1: Net-(D3-K) -> Net-(D3-Pad1)
- J2 pad 11: unconnected-(J2-GPIO1_B0-Pad11) -> /OrangePi 5 pro Header/STATUS LED
- J2 pad 23: unconnected-(J2-GPIO4_A7/I2C5_SDA-Pad23) -> /OrangePi 5 pro Header/USER LED 2
- J2 pad 24: unconnected-(J2-GPIO1_D7/I2C8_SDA/PWM15-Pad24) -> /OrangePi 5 pro Header/USER LED 1
- J2 pad 25: unconnected-(J2-GPIO1_A6-Pad25) -> /OrangePi 5 pro Header/USER BUTTON
- J2 pad 26: unconnected-(J2-GPIO1_A4-Pad26) -> /OrangePi 5 pro Header/ON OFF BTN
- J2 pad 34: /OrangePi 5 pro Header/GPIO4_B3/PWM15/CAN1_TX -> /Can Transiver/CAN_TR.TXD
- J2 pad 35: /OrangePi 5 pro Header/GPIO4_B2/PWM14/CAN1_RX -> /Can Transiver/CAN_TR.RXD
- J2 pad 4: unconnected-(J2-GPIO0_B5/UART2_TX-Pad4) -> /CH340_DEBUG/UART_DEBUG.TX
- J2 pad 43: /OrangePi 5 pro Header/USB20_DP4 -> /OrangePi 5 pro Header/USB_SBC.+
- J2 pad 44: /OrangePi 5 pro Header/USB20_DM4 -> /OrangePi 5 pro Header/USB_SBC.-
- J2 pad 47: /OrangePi 5 pro Header/USB20_DM3 -> /DIN41612 connector/USB_DEBUG.-
- J2 pad 48: /OrangePi 5 pro Header/USB20_DP3 -> /DIN41612 connector/USB_DEBUG.+
- J2 pad 5: unconnected-(J2-GPIO0_B6/UART2_RX-Pad5) -> /CH340_DEBUG/UART_DEBUG.RX
- J2 pad 6: unconnected-(J2-GPIO1_A7/PWM3-Pad6) -> /FAN controller/FAN_PWM
- L1 pad 1: Net-(U6-Lx) -> Net-(U2-Lx)
- Q1 pad 2: GND -> +5V
- Q1 pad 3: Net-(M1--) -> /Power Oring/BUCK_IN
- Q2 pad 1: Net-(Q2-G) -> /Power Oring/BUCK_IN
- Q2 pad 2: +5V -> GND
- Q2 pad 3: /5v buck/5V_OUT -> Net-(Q2-C)
- Q4 pad 1: /5v buck/5V_OUT -> Net-(Q4-G)
- Q4 pad 3: Net-(Q4-C) -> Net-(M1--)
- R1 pad 1: Net-(U1-VOUTL) -> /DIN41612 connector/12v
- R1 pad 2: Net-(C11-Pad1) -> Net-(U2-EN)
- R10 pad 1: Net-(M1-+) -> /USB-CAN/WORD_LED1
- R10 pad 2: +12V -> Net-(D2-Pad1)
- R11 pad 1: Net-(M1-+) -> /USB-CAN/STAT_LED1
- R11 pad 2: +5V -> Net-(D3-Pad1)
- R12 pad 1: GND -> /Power Oring/BUCK_IN
- R12 pad 2: Net-(Q1-G) -> Net-(Q2-C)
- R13 pad 1: /FAN controller/FAN_PWM -> /DIN41612 connector/5v_STDBY
- R13 pad 2: Net-(Q1-G) -> Net-(U5-EN)
- R14 pad 1: /DIN41612 connector/12v -> Net-(U6-STB)
- R14 pad 2: Net-(U6-EN) -> GND
- R15 pad 1: /5v buck/5V_OUT -> Net-(U7-STB)
- R15 pad 2: Net-(U6-FB) -> GND
- R16 pad 1: Net-(U6-EN) -> Net-(U9-VOUTL)
- R16 pad 2: GND -> Net-(C40-Pad1)
- R17 pad 1: Net-(U6-FB) -> Net-(U9-VOUTR)
- R17 pad 2: GND -> Net-(C40-Pad1)
- R18 pad 1: /5v buck/5V_OUT -> GND
- R18 pad 2: Net-(Q4-C) -> Net-(C40-Pad1)
- R19 pad 1: +3V3 -> +5V
- R19 pad 2: /USB-CAN/NRST1 -> /Audio Codec/USB_AUDIO.+
- R2 pad 1: Net-(U1-VOUTR) -> /5v buck/5V_OUT
- R2 pad 2: Net-(C11-Pad1) -> Net-(U2-FB)
- R20 pad 1: /USB-CAN/WORD_LED1 -> /Audio Codec/USB_AUDIO.+
- R20 pad 2: Net-(D2-K) -> /Audio Codec/D+
- R21 pad 1: /USB-CAN/STAT_LED1 -> /Audio Codec/USB_AUDIO.-
- R21 pad 2: Net-(D3-K) -> /Audio Codec/D-
- R22 pad 1: /DIN41612 connector/5v_STDBY -> Net-(U9-DT)
- R22 pad 2: Net-(U8-EN) -> +5V
- R3 pad 1: GND -> Net-(U2-EN)
- R3 pad 2: Net-(C11-Pad1) -> GND
- R4 pad 1: Net-(U1-DT) -> Net-(U2-FB)
- R4 pad 2: +5V -> GND
- R5 pad 1: +5V -> +3V3
- R5 pad 2: /Audio Codec/USB_AUDIO.+ -> /USB-CAN/NRST1
- R6 pad 1: /Audio Codec/USB_AUDIO.+ -> /USB-CAN/WORD_LED1
- R6 pad 2: /Audio Codec/D+ -> Net-(D1-Pad1)
- R7 pad 1: /Audio Codec/USB_AUDIO.- -> /USB-CAN/STAT_LED1
- R7 pad 2: /Audio Codec/D- -> Net-(D2-Pad1)
- R8 pad 1: GND -> /5v buck/5V_OUT
- R8 pad 2: Net-(U4-STB) -> Net-(Q2-C)
- R9 pad 1: GND -> +3V3
- R9 pad 2: Net-(U5-STB) -> /USB-CAN/NRST1
- RV1 pad 1: Net-(U2-V) -> Net-(U8-V)
- RV1 pad 2: Net-(U2-V) -> Net-(U8-V)
- U10 pad 1: /DIN41612 connector/USB1U.D- -> /Audio Codec/USB_AUDIO.-
- U10 pad 2: unconnected-(U10-VN-Pad2) -> /Audio Codec/USB_AUDIO.+
- U10 pad 3: /DIN41612 connector/USB1U.D- -> /USB HUB/USB_CAN.-
- U10 pad 4: /DIN41612 connector/USB1U.D+ -> /USB HUB/USB_CAN.+
- U10 pad 5: unconnected-(U10-VP-Pad5) -> /USB HUB/USB3.-
- U10 pad 6: /DIN41612 connector/USB1U.D+ -> /USB HUB/USB3.+
- U3 pad 1: /Audio Codec/USB_AUDIO.- -> +3V3
- U3 pad 10: /OrangePi 5 pro Header/USB_SBC.- -> unconnected-(U3-PA2-Pad10)
- U3 pad 11: /OrangePi 5 pro Header/USB_SBC.+ -> unconnected-(U3-PA3-Pad11)
- U3 pad 12: +5V -> unconnected-(U3-PA4-Pad12)
- U3 pad 13: Net-(U3-VDD33) -> unconnected-(U3-PA5-Pad13)
- U3 pad 14: GND -> unconnected-(U3-PA6-Pad14)
- U3 pad 15: Net-(U3-XO) -> unconnected-(U3-PA7-Pad15)
- U3 pad 16: Net-(U3-XI) -> unconnected-(U3-PB0-Pad16)
- U3 pad 2: /Audio Codec/USB_AUDIO.+ -> unconnected-(U3-PC13-Pad2)
- U3 pad 3: /USB HUB/USB_CAN.- -> unconnected-(U3-PC14-Pad3)
- U3 pad 4: /USB HUB/USB_CAN.+ -> unconnected-(U3-PC15-Pad4)
- U3 pad 5: /USB HUB/USB3.- -> unconnected-(U3-PF0-Pad5)
- U3 pad 6: /USB HUB/USB3.+ -> unconnected-(U3-PF1-Pad6)
- U3 pad 7: /USB HUB/USB4.- -> /USB-CAN/NRST1
- U3 pad 8: /USB HUB/USB4.+ -> /USB-CAN/LED_TX
- U3 pad 9: unconnected-(U3-RESET#/CDP-Pad9) -> /USB-CAN/LED_RX
- U4 pad 1: /Can Transiver/CAN_TR.TXD -> Net-(U4-VCAP)
- U4 pad 3: +5V -> Net-(Q2-C)
- U4 pad 4: /Can Transiver/CAN_TR.RXD -> +5V
- U4 pad 5: +3V3 -> Net-(Q1-G)
- U4 pad 6: /Can Transiver/CAN_TR_OUT.- -> /Power Oring/BUCK_IN
- U5 pad 1: /Can Transiver1/CAN_TR.TXD -> Net-(U5-VCAP)
- U5 pad 3: +5V -> Net-(U5-EN)
- U5 pad 4: /Can Transiver1/CAN_TR.RXD -> +5V
- U5 pad 5: +3V3 -> Net-(Q3-G)
- U5 pad 6: /Can Transiver1/CAN_TR_OUT.- -> /DIN41612 connector/5v_STDBY
- U6 pad 1: Net-(U6-BST) -> /Can Transiver/CAN_TR.TXD
- U6 pad 2: Net-(U6-Lx) -> GND
- U6 pad 3: Net-(U6-EN) -> +5V
- U6 pad 4: Net-(U6-SS) -> /Can Transiver/CAN_TR.RXD
- U6 pad 5: Net-(U6-FB) -> +3V3
- U6 pad 6: Net-(U6-VCC) -> /Can Transiver/CAN_TR_OUT.-
- U6 pad 7: /DIN41612 connector/12v -> /Can Transiver/CAN_TR_OUT.+
- U6 pad 8: /DIN41612 connector/12v -> Net-(U6-STB)
- U7 pad 1: Net-(U7-VCAP) -> /Can Transiver1/CAN_TR.TXD
- U7 pad 3: Net-(Q4-C) -> +5V
- U7 pad 4: +5V -> /Can Transiver1/CAN_TR.RXD
- U7 pad 5: Net-(Q2-G) -> +3V3
- U7 pad 6: /5v buck/5V_OUT -> /Can Transiver1/CAN_TR_OUT.-
- X1 pad 1: Net-(U1-XTI) -> Net-(U9-XTI)
- X1 pad 3: Net-(U1-XTO) -> Net-(U9-XTO)
- Y1 pad 1: Net-(U3-XI) -> Net-(U10-XI)
- Y1 pad 3: Net-(U3-XO) -> Net-(U10-XO)
Other:
- board outline removed

Commit message: Figure out SSPND pin
Parts:
- removed C16, C17: 1uF, PCM_JLCPCB:C_0402
- removed D1: Green, PCM_JLCPCB:D_0603
- removed L1: 6.8uH 12.5x12.5mm, Inductor_SMD:L_AVX_LMLP07A7
- removed Q2: MMBT3904, PCM_JLCPCB:Q_SOT-23
- added C57: 22uF, PCM_JLCPCB:C_0805, F.Cu at (220.6, 107.4)
- added C58: 22uF, PCM_JLCPCB:C_0805, F.Cu at (220.6, 110.4)
- added JP1: Solder Jumper, Jumper:SolderJumper-2_P1.3mm_Open_RoundedPad1.0x1.5mm, F.Cu at (225.0, 107.7)
- added L2: 1uH, Inductor_SMD:L_Sunlord_MWSA1005S, F.Cu at (225.9, 100.1)
- added LED2: FixLed307, FixLed307:FixLed307, F.Cu at (238.4, 100.8)
- added Q5: MMBT3904, PCM_JLCPCB:Q_SOT-23, F.Cu at (237.9, 109.9)
- added R32: 20kΩ, PCM_JLCPCB:R_0402, F.Cu at (224.2, 110.4)
- added R33: 1kΩ, PCM_JLCPCB:R_0402, F.Cu at (242.8, 95.2)
- added R34: 1kΩ, PCM_JLCPCB:R_0402, F.Cu at (242.8, 97.0)
- added R35: 1kΩ, PCM_JLCPCB:R_0402, F.Cu at (242.8, 98.9)
- C10: value 100nF 50V Y5V -> 22uF; footprint Capacitor_SMD:C_0402_1005Metric -> PCM_JLCPCB:C_0805
- C11: value 10uF -> 100nF; footprint PCM_JLCPCB:C_1206 -> PCM_JLCPCB:C_0402
- C12, C13: value 10uF -> 22uF; footprint PCM_JLCPCB:C_1206 -> PCM_JLCPCB:C_0805
- C14: value 10uF -> 1uF; footprint PCM_JLCPCB:C_1206 -> PCM_JLCPCB:C_0402
- C15: value 100nF 50V Y5V -> 4.7uF; footprint Capacitor_SMD:C_0402_1005Metric -> PCM_JLCPCB:C_0805
- C8: value 47uF -> 22uF; footprint Capacitor_SMD:CP_Elec_6.3x5.4 -> PCM_JLCPCB:C_0805
- C9: value 10uF 50v -> 100nF; footprint Capacitor_SMD:C_0805_2012Metric -> PCM_JLCPCB:C_0402
- R1: value 39k 1% -> 2.2kΩ; footprint Resistor_SMD:R_0402_1005Metric -> PCM_JLCPCB:R_0402
- R2: value 31.6k 1% -> 10kΩ; footprint Resistor_SMD:R_0402_1005Metric -> PCM_JLCPCB:R_0402
- R3: value 10k 1% -> 73k2; footprint Resistor_SMD:R_0402_1005Metric -> PCM_JLCPCB:R_0402
- R4: value 10k 1% -> R_499k_0402
- R5: value 10k -> 1kΩ; footprint Resistor_SMD:R_0402_1005Metric -> PCM_JLCPCB:R_0402
- R6: value 1k -> 10kΩ; footprint Resistor_SMD:R_0402_1005Metric -> PCM_JLCPCB:R_0402
- R7: value 1k -> R_499k_0402
- R8: value 10kΩ -> R_499k_0402; footprint PCM_JLCPCB:R_0402 -> Resistor_SMD:R_0402_1005Metric
Connections:
- net /Audio Codec/VCOM renamed Net-(U9-VCOM)
- net /Power Oring/BUCK_IN renamed /5v buck/BUCK_OUT
- C10 pad 1: /DIN41612 connector/12v -> /5v buck/V_{IN}
- C11 pad 1: /5v buck/5V_OUT -> /5v buck/V_{IN}
- C14 pad 1: /5v buck/5V_OUT -> /5v buck/5V_VDD
- C15 pad 1: /5v buck/5V_OUT -> /5v buck/5V_VDRV
- C34 pad 1: Net-(U9-VBUS) -> /Audio Codec/VDD_{int}
- C7 pad 1: Net-(U2-BST) -> /5v buck/5V_BOOT
- C7 pad 2: Net-(U2-Lx) -> /5v buck/5V_PHASE
- C8 pad 1: /DIN41612 connector/12v -> /5v buck/5V_OUT
- C9 pad 1: /DIN41612 connector/12v -> /5v buck/5V_EN
- J1 pad a11: /DIN41612 connector/12v -> /5v buck/V_{IN}
- J1 pad a12: /DIN41612 connector/12v -> /5v buck/V_{IN}
- J1 pad b11: /DIN41612 connector/12v -> /5v buck/V_{IN}
- J1 pad b12: /DIN41612 connector/12v -> /5v buck/V_{IN}
- J1 pad c11: /DIN41612 connector/12v -> /5v buck/V_{IN}
- J1 pad c12: /DIN41612 connector/12v -> /5v buck/V_{IN}
- LED1 pad 1: unconnected-(LED1-Pad1) -> /OrangePi 5 pro Header/STATUS LED
- LED1 pad 2: unconnected-(LED1-Pad2) -> Net-(LED1-Pad2)
- LED1 pad 3: unconnected-(LED1-Pad3) -> +5V
- LED1 pad 4: unconnected-(LED1-Pad4) -> Net-(LED1-Pad4)
- R1 pad 1: /DIN41612 connector/12v -> /5v buck/5V_EN
- R1 pad 2: Net-(U2-EN) -> GND
- R12 pad 2: Net-(Q2-C) -> Net-(U4-EN)
- R19 pad 1: +5V -> /Audio Codec/VDD_{int}
- R2 pad 1: /5v buck/5V_OUT -> /5v buck/5V_FB
- R2 pad 2: Net-(U2-FB) -> GND
- R22 pad 2: +5V -> /Audio Codec/VDD_{int}
- R3 pad 1: Net-(U2-EN) -> /5v buck/5V_OUT
- R3 pad 2: GND -> /5v buck/5V_FB
- R4 pad 1: Net-(U2-FB) -> /5v buck/5V_MODE1
- R4 pad 2: GND -> /5v buck/5V_VDD
- R5 pad 1: +3V3 -> Net-(LED1-Pad4)
- R5 pad 2: /USB-CAN/NRST1 -> GND
- R6 pad 1: /USB-CAN/WORD_LED1 -> /5v buck/5V_OUT
- R6 pad 2: Net-(D1-Pad1) -> /5v buck/Pgood
- R7 pad 1: /USB-CAN/STAT_LED1 -> GND
- R7 pad 2: Net-(D2-Pad1) -> /5v buck/5V_MODE1
- R8 pad 1: /5v buck/5V_OUT -> GND
- R8 pad 2: Net-(Q2-C) -> /5v buck/5V_MODE2
- U4 pad 3: Net-(Q2-C) -> Net-(U4-EN)

Commit message: Prepare board for layout
Parts:
- removed J4: Connector, USB-TYPE-C-16P, USB_C_Upright16pin:MOLEX_2169890001
- removed Q3: AO3400, Package_TO_SOT_SMD:SOT-23
- removed R19: 1.5kΩ, PCM_JLCPCB:R_0402
- added C16: 100nF, PCM_JLCPCB:C_0402, F.Cu at (172.6, 35.8)
- added C17: 100nF, PCM_JLCPCB:C_0402, F.Cu at (135.8, 63.8)
- added C59: 100nF, PCM_JLCPCB:C_0402, F.Cu at (135.8, 78.6)
- added C60: 100nF, PCM_JLCPCB:C_0402, F.Cu at (172.6, 37.6)
- added J5: Connector, USB-TYPE-C-16P, PCM_JLCPCB:TYPE-C-SMD_HX-TYPE-C-16PIN, F.Cu at (144.2, 45.5)
- added Q2: AO3400A, Package_TO_SOT_SMD:SOT-23, F.Cu at (182.0, 126.6)
- added R36: 499k, PCM_JLCPCB:R_0402, F.Cu at (214.9, 131.5)
- added R37: 100Ω, PCM_JLCPCB:R_0402, F.Cu at (169.5, 39.8)
- added R38: 10kΩ, PCM_JLCPCB:R_0402, F.Cu at (169.5, 41.6)
- added R39: 10kΩ, PCM_JLCPCB:R_0402, F.Cu at (169.5, 43.5)
- added R40: 20kΩ, PCM_JLCPCB:R_0402, F.Cu at (120.6, 93.1)
- added R41: 10kΩ, PCM_JLCPCB:R_0402, F.Cu at (120.6, 95.0)
- added R42: 1.5kΩ, PCM_JLCPCB:R_0603, F.Cu at (97.0, 61.2)
- added U13: AMS1117-3.3, Package_TO_SOT_SMD:SOT-223-3_TabPin2, F.Cu at (175.8, 107.0)
- added U8: TDA7052A, Package_SO:SO-8_3.9x4.9mm_P1.27mm, F.Cu at (79.0, 63.5)
- added U9: PCM2704CDBR, PCM2704:SOP65P780X200-28N, F.Cu at (96.0, 67.5)
- Q1: value AO3400 -> AO3400A
- R20, R21: value 22Ω -> 0Ω
- R4, R7: value R_499k_0402 -> 499k; footprint Resistor_SMD:R_0402_1005Metric -> PCM_JLCPCB:R_0402
- R8: value R_499k_0402 -> 100Ω; footprint Resistor_SMD:R_0402_1005Metric -> PCM_JLCPCB:R_0402
- RV1: value 1Meg Bourns 3296 -> RM065 1Meg; footprint Potentiometer_THT:Potentiometer_Bourns_3296W_Vertical -> Potentiometer_THT:Potentiometer_Runtron_RM-065_Vertical
- U2: value ~ -> SIC431AED-T1-GE3; footprint Package_SO:Diodes_SO-8EP -> SIC471:REGULATOR_SIC431AED-T1-GE3
- moved C34 126.7 mm to (25.4, 54.6)
- moved C35 126.7 mm to (25.4, 56.4)
- moved C39 126.7 mm to (28.3, 54.6)
- moved C32 126.7 mm to (25.4, 52.7)
- moved C36 126.7 mm to (25.4, 58.3)
- moved C38 126.7 mm to (28.3, 52.7)
- moved LED2 126.0 mm to (125.6, 44.9)
- moved D4 116.2 mm to (94.2, 117.8), turned to 90 degrees
- moved X1 107.7 mm to (38.9, 84.0)
- moved C33 107.7 mm to (34.1, 83.6)
- moved C37 107.7 mm to (34.1, 86.6)
- moved C50 103.7 mm to (89.2, 118.5), turned to 90 degrees
- moved R22 101.6 mm to (98.8, 62.2), turned to 180 degrees
- moved C8 97.7 mm to (224.3, 148.1), turned to 180 degrees
- moved C49 97.0 mm to (105.2, 118.5)
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Connections:
- net /Can Transiver/CAN_TR_OUT.+ renamed /Can Transiver/CAN_TR_OUT.C+
- net /Can Transiver/CAN_TR_OUT.- renamed /Can Transiver/CAN_TR_OUT.C-
- net /Can Transiver1/CAN_TR_OUT.+ renamed /Can Transiver1/CAN_TR_OUT.C+
- net /Can Transiver1/CAN_TR_OUT.- renamed /Can Transiver1/CAN_TR_OUT.C-
- net /DIN41612 connector/GPIOR14 renamed /DIN41612 connector/USB_IN.D-
- net /DIN41612 connector/GPIOR15 renamed /DIN41612 connector/USB_IN.D+
- net /Panel USB/USB_IN.+ renamed /Panel USB/USB_IN.D+
- net /Panel USB/USB_IN.- renamed /Panel USB/USB_IN.D-
- net /USB HUB/USB3.+ renamed /USB HUB/USB3.D+
- net /USB HUB/USB3.- renamed /USB HUB/USB3.D-
- net /USB HUB/USB4.+ renamed /USB HUB/USB4.D+
- net /USB HUB/USB4.- renamed /USB HUB/USB4.D-
- BTN1 pad 1: unconnected-(BTN1-Pad1) -> GND
- BTN1 pad 2: unconnected-(BTN1-Pad2) -> GND
- BTN1 pad 3: /OrangePi 5 pro Header/USER BUTTON -> Net-(BTN1-Pad3)
- BTN1 pad 4: /OrangePi 5 pro Header/ON OFF BTN -> Net-(BTN1-Pad4)
- C35 pad 1: Net-(U9-VCCL) -> /Audio Codec/VCCL
- C38 pad 1: Net-(U9-VCCR) -> /Audio Codec/VCCR
- C39 pad 1: Net-(U9-VCCP) -> /Audio Codec/VCCP
- J1 pad a2: /DIN41612 connector/USB1U.D+ -> unconnected-(J1-Pada2)
- J1 pad c2: /DIN41612 connector/USB1U.D- -> unconnected-(J1-Padc2)
- J2 pad 22: unconnected-(J2-GPIO4_A6/UART3_RX/I2C5_SCL-Pad22) -> Net-(J2-GPIO4_A6/UART3_RX/I2C5_SCL)
- J2 pad 43: /OrangePi 5 pro Header/USB_SBC.+ -> /DIN41612 connector/USB_DEBUG.D+
- J2 pad 44: /OrangePi 5 pro Header/USB_SBC.- -> /DIN41612 connector/USB_DEBUG.D-
- J2 pad 47: /DIN41612 connector/USB_DEBUG.- -> /OrangePi 5 pro Header/USB_OUT.D-
- J2 pad 48: /DIN41612 connector/USB_DEBUG.+ -> /OrangePi 5 pro Header/USB_OUT.D+
- LED1 pad 3: +5V -> +3V3
- Q1 pad 2: +5V -> /DIN41612 connector/5v_STDBY
- Q1 pad 3: /5v buck/BUCK_OUT -> +5V
- R10 pad 1: /USB-CAN/WORD_LED1 -> /USB-CAN/LED_RX
- R11 pad 1: /USB-CAN/STAT_LED1 -> /USB-CAN/LED_TX
- R20 pad 1: /Audio Codec/USB_AUDIO.+ -> /CH340_DEBUG/TXD
- R20 pad 2: /Audio Codec/D+ -> /CH340_DEBUG/UART_DEBUG.RX
- R21 pad 1: /Audio Codec/USB_AUDIO.- -> /CH340_DEBUG/RXD
- R21 pad 2: /Audio Codec/D- -> /CH340_DEBUG/UART_DEBUG.TX
- R23 pad 2: +12V -> /5v buck/V_{IN}
- R4 pad 1: /5v buck/5V_MODE1 -> /5v buck/5V_VDD
- R4 pad 2: /5v buck/5V_VDD -> /5v buck/5V_MODE1
- R7 pad 1: GND -> /5v buck/5V_MODE2
- R7 pad 2: /5v buck/5V_MODE1 -> GND
- R8 pad 1: GND -> Net-(BTN1-Pad3)
- R8 pad 2: /5v buck/5V_MODE2 -> /OrangePi 5 pro Header/USER BUTTON
- U1 pad 3: /DIN41612 connector/USB_DEBUG.- -> /DIN41612 connector/USB_DEBUG.D-
- U1 pad 4: /DIN41612 connector/USB_DEBUG.+ -> /DIN41612 connector/USB_DEBUG.D+
- U10 pad 1: /Audio Codec/USB_AUDIO.- -> /USB HUB/USB_CAN.D-
- U10 pad 10: /OrangePi 5 pro Header/USB_SBC.- -> /OrangePi 5 pro Header/USB_OUT.D-
- U10 pad 11: /OrangePi 5 pro Header/USB_SBC.+ -> /OrangePi 5 pro Header/USB_OUT.D+
- U10 pad 2: /Audio Codec/USB_AUDIO.+ -> /USB HUB/USB_CAN.D+
- U10 pad 3: /USB HUB/USB_CAN.- -> /Audio Codec/USB_AUDIO.D-
- U10 pad 4: /USB HUB/USB_CAN.+ -> /Audio Codec/USB_AUDIO.D+
- U11 pad 2: /CH340_DEBUG/UART_DEBUG.RX -> /CH340_DEBUG/TXD
- U11 pad 3: /CH340_DEBUG/UART_DEBUG.TX -> /CH340_DEBUG/RXD
- U12 pad 3: /Panel USB/FRONT_PANEL.D- -> /CH340_DEBUG/FRONT_PANEL.D+
- U12 pad 4: /Panel USB/FRONT_PANEL.D+ -> /CH340_DEBUG/FRONT_PANEL.D-
- U2 pad 1: Net-(U2-BST) -> /5v buck/V_{IN}
- U2 pad 2: Net-(U2-Lx) -> /5v buck/V_{IN}
- U2 pad 3: Net-(U2-EN) -> GND
- U2 pad 4: Net-(U2-SS) -> GND
- U2 pad 5: Net-(U2-FB) -> /5v buck/5V_SW
- U2 pad 6: Net-(U2-VCC) -> /5v buck/5V_SW
- U2 pad 7: /DIN41612 connector/12v -> /5v buck/5V_SW
- U2 pad 8: /DIN41612 connector/12v -> /5v buck/5V_SW
- U2 pad 9: GND -> /5v buck/5V_SW
- U3 pad 33: /USB HUB/USB_CAN.- -> /USB HUB/USB_CAN.D-
- U3 pad 34: /USB HUB/USB_CAN.+ -> /USB HUB/USB_CAN.D+
- U4 pad 5: Net-(Q1-G) -> Net-(Q2-G)
- U5 pad 5: Net-(Q3-G) -> Net-(Q1-G)
Routing:
- net /Can Transiver/CAN_TR.TXD: track 0.00 -> 7.63 mm
- net /Can Transiver/CAN_TR.RXD: track 0.00 -> 7.58 mm
- net Net-(J5-D--PadA7): track 0.00 -> 4.49 mm
- net Net-(J5-D+-PadA6): track 0.00 -> 4.49 mm
- net /CH340_DEBUG/RXD: track 0.00 -> 3.63 mm
- net Net-(U11-XI): track 0.00 -> 3.20 mm
- net /Can Transiver1/CAN_TR.TXD: track 0.00 -> 2.71 mm
- net /DIN41612 connector/USB_DEBUG.D-: track 0.00 -> 2.59 mm
- net /Can Transiver1/CAN_TR.RXD: track 0.00 -> 2.57 mm
- net /CH340_DEBUG/TXD: track 0.00 -> 2.51 mm
- net /Panel USB/USB_IN.D-: track 0.00 -> 1.89 mm
- net /Panel USB/USB_IN.D+: track 0.00 -> 1.89 mm
- net /DIN41612 connector/USB_DEBUG.D+: track 0.00 -> 1.20 mm
Other:
- board outline added: 100 x 100 mm
- board text added: "DON'T PUT ANYTHING HERE"

Commit message: Do buck Layout
Parts:
- removed R42: 1.5kΩ, PCM_JLCPCB:R_0603
- added C61: 10uF, PCM_JLCPCB:C_0603, F.Cu at (125.0, 109.0)
- added C62: 10uF, PCM_JLCPCB:C_0603, F.Cu at (125.0, 110.3)
- added C63: 10uF, PCM_JLCPCB:C_0603, F.Cu at (125.0, 111.6)
- added R19: 1.5kΩ, PCM_JLCPCB:R_0402, F.Cu at (25.5, 25.9)
- C12, C13, C58, C8: value 22uF -> 10uF; footprint PCM_JLCPCB:C_0805 -> PCM_JLCPCB:C_0603
- C15: footprint PCM_JLCPCB:C_0805 -> PCM_JLCPCB:C_0402
- L2: footprint Inductor_SMD:L_Sunlord_MWSA1005S -> Inductor_SMD:L_Bourns_SRP7028A_7.3x6.6mm
- moved Y1 112.9 mm to (119.0, 23.9)
- moved C41 112.1 mm to (42.1, 31.6)
- moved C10 101.9 mm to (128.2, 111.2)
- moved C8 100.6 mm to (129.7, 113.8), turned to 90 degrees
- moved C13 100.4 mm to (127.1, 113.8), turned to 90 degrees
- moved C12 100.0 mm to (128.4, 113.8), turned to 90 degrees
- moved C58 99.8 mm to (125.8, 113.8), turned to 90 degrees
- moved C57 99.0 mm to (128.2, 109.2)
- moved C9 94.1 mm to (131.0, 106.4)
- moved C11 93.6 mm to (130.5, 108.0), turned to 90 degrees
- moved C7 92.9 mm to (131.9, 109.6)
- moved C15 90.8 mm to (136.3, 113.8), turned to 90 degrees
- moved R1 90.3 mm to (132.3, 108.0), turned to -90 degrees
- moved JP1 89.5 mm to (123.4, 113.7)
- moved C1 89.0 mm to (138.8, 120.2), turned to 90 degrees
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Connections:
- J2 pad 32: +3V3 -> unconnected-(J2-3V3-Pad32)
- J2 pad 40: +3V3 -> unconnected-(J2-3V3-Pad40)
- U2 pad 27_1: (no net) -> GND
- U2 pad 27_2: (no net) -> GND
- U2 pad 9.1: (no net) -> /5v buck/5V_SW
Routing:
- net Net-(Q2-G): track 0.00 -> 9.86 mm, vias 0 -> 2
- net /DIN41612 connector/5v_STDBY: track 0.00 -> 8.87 mm
- net Net-(Q1-G): track 0.00 -> 8.57 mm
- net /5v buck/5V_EN: track 0.00 -> 8.30 mm, vias 0 -> 2
- net /Can Transiver/CAN_TR.TXD: track 7.63 -> 0.00 mm
- net /Can Transiver/CAN_TR.RXD: track 7.58 -> 0.00 mm
- net /5v buck/BUCK_OUT: track 0.00 -> 5.66 mm
- net Net-(U10-XI): track 0.00 -> 4.13 mm
- net Net-(U11-XO): track 0.00 -> 4.02 mm
- net Net-(U10-VDD33): track 0.00 -> 4.00 mm
- net /5v buck/5V_MODE1: track 0.00 -> 3.71 mm
- net /CH340_DEBUG/RXD: track 3.63 -> 0.00 mm
- net Net-(U10-XO): track 0.00 -> 3.39 mm
- net Net-(BTN1-Pad3): track 0.00 -> 3.22 mm
- net Net-(BTN1-Pad4): track 0.00 -> 3.13 mm
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- added copper zone on F.Cu, net +3V3
- added copper zone on F.Cu, net +5V
- added copper zone on F.Cu, net /5v buck/5V_EN
- added copper zone on F.Cu, net /5v buck/5V_OUT
- added copper zone on F.Cu, net /5v buck/5V_SW
- added copper zone on F.Cu, net /5v buck/BUCK_OUT
- added copper zone on F.Cu, net /5v buck/V_{IN}
- added copper zone on F.Cu, net /DIN41612 connector/5v_STDBY
- added copper zone on F.Cu, net GND
- added copper zone on F.Cu, net Net-(M1-+)
- added copper zone on F.Cu, net Net-(M1--)
