File: PCB source/5v buck.kicad_sch (KiCad schematic)
At the start: 22 parts, among them U2 SIC431AED-T1-GE3

Commit message: Pass ERC
Parts:
- removed R4, R7, R8: R_499k_0402, Resistor_SMD:R_0402_1005Metric, symbol antmicroResistors0402:R_499k_0402
- added R36, R4, R7: 499k, PCM_JLCPCB:R_0402, symbol PCM_JLCPCB-Resistors:0402,0Ω
- U2: footprint antmicro-footprints:MLP44-24L_4x4x0.75mm -> SIC471:REGULATOR_SIC431AED-T1-GE3
Connections:
- net 5V_MODE1: now also R36.1, R4.2
- net 5V_MODE2: now also R7.1
- net 5V_VDD: now also R4.1
- net GND: now also R36.2, R7.2

Commit message: Do buck Layout
Parts:
- removed C12, C13, C58, C8: 22uF, PCM_JLCPCB:C_0805, symbol PCM_JLCPCB-Capacitors:0805,22uF
- removed C15: 4.7uF, PCM_JLCPCB:C_0805, symbol PCM_JLCPCB-Capacitors:0805,4.7uF
- added C12, C13, C58, C61, C62, C63, C8: 10uF, PCM_JLCPCB:C_0603, symbol PCM_JLCPCB-Capacitors:0603,10uF
- added C15: 4.7uF, PCM_JLCPCB:C_0402, symbol PCM_JLCPCB-Capacitors:0402,4.7uF
- L2: footprint Inductor_SMD:L_Sunlord_MWSA1005S -> Inductor_SMD:L_Bourns_SRP7028A_7.3x6.6mm
Connections:
- net 5V_OUT: now also C12.1, C13.1, C58.1, C61.1, C62.1, C63.1, C8.1
- net 5V_SW: now also U2.9.1 (SW)
- net 5V_VDRV: now also C15.1
- net GND: now also U2.27_1 (GND), U2.27_2 (GND), C12.2, C13.2, C15.2, C58.2, C61.2, C62.2, C63.2, C8.2
Other:
- moved on the sheet: C10, C11, C14, C57, C7, C9, JP1, L2, R1, R2, R3, R32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

Commit message: Fix schematic
Parts:
- C10, C57: Price 0.024USD -> 0.026USD; Stock 2916538 -> 2530414
- C11, C7, C9: Stock 5358037 -> 5436546
- C12, C13, C58, C61, C62, C63, C8: Stock 11848478 -> 8972925
- C14: Stock 8324208 -> 6453835
- C15: Stock 846222 -> 1633861
- R1: Stock 1186966 -> 2234263
- R2, R6: Stock 6666349 -> 13746052
- R3: Stock 5514860 -> 6249348
- R32: Stock 1747699 -> 1163119
- R36, R4, R7: LCSC (none) -> C17168; Stock (none) -> 6249348
