File: PCB source/CH340_DEBUG.kicad_sch (KiCad schematic)
At the start: 6 parts, among them U11 CH340G, Y2 12MHz C7424717

Commit message: Do Cleanup
Parts:
- renumbered C50 to C51, C51 to C52, C52 to C53, C53 to C54
Changed lines of the file:
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@@
 		(on_board yes)
 		(dnp no)
-		(property "Reference" "C53"
+		(property "Reference" "C54"
 			(at 115.57 125.7362 0)
 			(effects
@@
 			(project "OrangePie"
 				(path "/3103c9de-f1ba-4d51-8bfc-798df1c75e2f/6795f84c-4c2f-4fb2-bd1b-dc83d61d75c6"
-					(reference "C53")
+					(reference "C54")
 					(unit 1)
 				)
@@
 		(on_board yes)
 		(dnp no)
-		(property "Reference" "C52"
+		(property "Reference" "C53"
 			(at 97.79 125.7362 0)
 			(effects
@@
 			(project "OrangePie"
 				(path "/3103c9de-f1ba-4d51-8bfc-798df1c75e2f/6795f84c-4c2f-4fb2-bd1b-dc83d61d75c6"
-					(reference "C52")
+					(reference "C53")
 					(unit 1)
 				)
@@
 		(on_board yes)
 		(dnp no)
-		(property "Reference" "#PWR087"
+		(property "Reference" "#PWR0107"
 			(at 105.41 118.11 0)
 			(effects
@@
 			(project "OrangePie"
 				(path "/3103c9de-f1ba-4d51-8bfc-798df1c75e2f/6795f84c-4c2f-4fb2-bd1b-dc83d61d75c6"
-					(reference "#PWR087")
+					(reference "#PWR0107")
 					(unit 1)
 				)
@@
 		(dnp no)
 		(fields_autoplaced yes)
-		(property "Reference" "#PWR078"
+		(property "Reference" "#PWR0104"
 			(at 130.81 73.66 0)
 			(effects
@@
 			(project "OrangePie"
 				(path "/3103c9de-f1ba-4d51-8bfc-798df1c75e2f/6795f84c-4c2f-4fb2-bd1b-dc83d61d75c6"
-					(reference "#PWR078")
+					(reference "#PWR0104")
 					(unit 1)
 				)
@@
 		(dnp no)
 		(fields_autoplaced yes)
-		(property "Reference" "C51"
+		(property "Reference" "C52"
 			(at 154.94 80.01 0)
 			(effects
@@
 			(project "OrangePie"
 				(path "/3103c9de-f1ba-4d51-8bfc-798df1c75e2f/6795f84c-4c2f-4fb2-bd1b-dc83d61d75c6"
-					(reference "C51")
+					(reference "C52")
 					(unit 1)
 				)
@@
 		(on_board yes)
 		(dnp no)
-		(property "Reference" "#PWR099"
+		(property "Reference" "#PWR0111"
 			(at 133.35 137.16 0)
 			(effects
@@
 			(project "OrangePie"
 				(path "/3103c9de-f1ba-4d51-8bfc-798df1c75e2f/6795f84c-4c2f-4fb2-bd1b-dc83d61d75c6"
-					(reference "#PWR099")
+					(reference "#PWR0111")
 					(unit 1)
 				)
@@
 		(on_board yes)
 		(dnp no)
-		(property "Reference" "#PWR085"
+		(property "Reference" "#PWR0105"
 			(at 111.76 92.71 0)
 			(effects
@@
 			(project "OrangePie"
 				(path "/3103c9de-f1ba-4d51-8bfc-798df1c75e2f/6795f84c-4c2f-4fb2-bd1b-dc83d61d75c6"
-					(reference "#PWR085")
+					(reference "#PWR0105")
 					(unit 1)
 				)
@@
 		(dnp no)
 		(fields_autoplaced yes)
-		(property "Reference" "C50"
+		(property "Reference" "C51"
 			(at 114.3 80.01 0)
 			(effects
@@
 			(project "OrangePie"
 				(path "/3103c9de-f1ba-4d51-8bfc-798df1c75e2f/6795f84c-4c2f-4fb2-bd1b-dc83d61d75c6"
-					(reference "C50")
+					(reference "C51")
 					(unit 1)
 				)
@@
 		(on_board yes)
 		(dnp no)
-		(property "Reference" "#PWR091"
+		(property "Reference" "#PWR0109"
 			(at 109.22 137.16 0)
 			(effects
@@
 			(project "OrangePie"
 				(path "/3103c9de-f1ba-4d51-8bfc-798df1c75e2f/6795f84c-4c2f-4fb2-bd1b-dc83d61d75c6"
-					(reference "#PWR091")
+					(reference "#PWR0109")
 					(unit 1)
 				)
@@
 		(on_board yes)
 		(dnp no)
-		(property "Reference" "#PWR092"
+		(property "Reference" "#PWR0110"
 			(at 118.11 137.16 0)
 			(effects
@@
 			(project "OrangePie"
 				(path "/3103c9de-f1ba-4d51-8bfc-798df1c75e2f/6795f84c-4c2f-4fb2-bd1b-dc83d61d75c6"
-					(reference "#PWR092")
+					(reference "#PWR0110")
 					(unit 1)
 				)
@@
 		(on_board yes)
 		(dnp no)
-		(property "Reference" "#PWR086"
+		(property "Reference" "#PWR0106"
 			(at 152.4 92.71 0)
 			(effects
@@
 			(project "OrangePie"
 				(path "/3103c9de-f1ba-4d51-8bfc-798df1c75e2f/6795f84c-4c2f-4fb2-bd1b-dc83d61d75c6"
-					(reference "#PWR086")
+					(reference "#PWR0106")
 					(unit 1)
 				)
@@
 		(on_board yes)
 		(dnp no)
-		(property "Reference" "#PWR088"
+		(property "Reference" "#PWR0108"
 			(at 100.33 137.16 0)
 			(effects
@@
 			(project "OrangePie"
 				(path "/3103c9de-f1ba-4d51-8bfc-798df1c75e2f/6795f84c-4c2f-4fb2-bd1b-dc83d61d75c6"
-					(reference "#PWR088")
-					(unit 1)
-				)
+					(reference "#PWR0108")
+					(unit 1)
+				)

Commit message: Pass ERC
Connections:
- net FRONT_PANEL.D+ renamed FRONT_PANEL.+
- net FRONT_PANEL.D- renamed FRONT_PANEL.-
- net RXD renamed UART_DEBUG.TX
- net TXD renamed UART_DEBUG.RX
- no-connect marks 1 -> 7
Changed lines of the file:
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@@
+	)
+	(no_connect
+		(at 143.51 109.22)
+	)
+	(no_connect
+		(at 143.51 101.6)
+	)
+	(no_connect
+		(at 143.51 99.06)
+	)
+	(no_connect
+		(at 143.51 106.68)
+	)
+	(no_connect
+		(at 143.51 104.14)
 	)
 	(no_connect
 		(at 123.19 93.98)
+	)
+	(no_connect
+		(at 143.51 111.76)
 	)
 	(bus_entry
@@
 		)
 	)
-	(label "TXD"
-		(at 160.02 91.44 0)
-		(fields_autoplaced yes)
-		(effects
-			(font
-				(size 1.27 1.27)
-			)
-			(justify left bottom)
-		)
-	)
-	(label "RXD"
-		(at 160.02 93.98 0)
-		(fields_autoplaced yes)
-		(effects
-			(font
-				(size 1.27 1.27)
-			)
-			(justify left bottom)
-		)
-	)
 	(label "UART_DEBUG.RX"
 		(at 179.07 95.25 0)
@@
 		)
 	)
-	(label "FRONT_PANEL.D-"
+	(label "FRONT_PANEL.-"
 		(at 91.44 101.6 0)
 		(fields_autoplaced yes)
@@
 		)
 	)
-	(label "FRONT_PANEL.D+"
+	(label "FRONT_PANEL.+"
 		(at 91.44 99.06 0)
 		(fields_autoplaced yes)

Commit message: Prepare board for layout
Parts:
- added R20, R21: 0Ω, PCM_JLCPCB:R_0402, symbol PCM_JLCPCB-Resistors:0402,0Ω
Connections:
- net UART_DEBUG.RX: now also R20.2; no longer U11.2 (TXD)
- net UART_DEBUG.TX: now also R21.2; no longer U11.3 (RXD)
- net FRONT_PANEL.+ renamed FRONT_PANEL.D+
- net FRONT_PANEL.- renamed FRONT_PANEL.D-
- new net RXD: R21.1, U11.3 (RXD)
- new net TXD: R20.1, U11.2 (TXD)

Commit message: Fix schematic
Parts:
- C51, C52: Stock 5358037 -> 5436546
- R20, R21: Stock 5514860 -> 6249348
