File: PCB source/DIN41612 connector.kicad_sch (KiCad schematic)
At the start: 2 parts, among them J3 09031967921, U13 IP4234CZ6,115

Commit message: Do Cleanup
Parts:
- renumbered J3 to J1, U13 to U1
Changed lines of the file:
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@@
 	(label "USB_DEBUG.+"
 		(at 166.37 133.35 0)
+		(fields_autoplaced yes)
 		(effects
 			(font
@@
 	(label "CAN2_TR_OUT.+"
 		(at 200.66 74.93 0)
+		(fields_autoplaced yes)
 		(effects
 			(font
@@
 	(label "CAN2_TR_OUT.-"
 		(at 200.66 77.47 0)
+		(fields_autoplaced yes)
 		(effects
 			(font
@@
 	(label "USB_DEBUG.-"
 		(at 166.37 138.43 0)
+		(fields_autoplaced yes)
 		(effects
 			(font
@@
 		(on_board yes)
 		(dnp no)
-		(property "Reference" "#PWR098"
+		(property "Reference" "#PWR016"
 			(at 71.12 107.95 0)
 			(effects
@@
 			(project "OrangePie"
 				(path "/3103c9de-f1ba-4d51-8bfc-798df1c75e2f/50dedcd5-65c1-4d6e-8d03-473117f8d376"
-					(reference "#PWR098")
+					(reference "#PWR016")
 					(unit 1)
 				)
@@
 		(on_board yes)
 		(dnp no)
-		(property "Reference" "#PWR0107"
+		(property "Reference" "#PWR022"
 			(at 71.12 140.97 0)
 			(effects
@@
 			(project "OrangePie"
 				(path "/3103c9de-f1ba-4d51-8bfc-798df1c75e2f/50dedcd5-65c1-4d6e-8d03-473117f8d376"
-					(reference "#PWR0107")
+					(reference "#PWR022")
 					(unit 1)
 				)
@@
 		(on_board yes)
 		(dnp no)
-		(property "Reference" "#PWR079"
+		(property "Reference" "#PWR03"
 			(at 69.85 29.21 0)
 			(effects
@@
 			(project "OrangePie"
 				(path "/3103c9de-f1ba-4d51-8bfc-798df1c75e2f/50dedcd5-65c1-4d6e-8d03-473117f8d376"
-					(reference "#PWR079")
+					(reference "#PWR03")
 					(unit 1)
 				)
@@
 		(on_board yes)
 		(dnp no)
-		(property "Reference" "#PWR083"
+		(property "Reference" "#PWR07"
 			(at 69.85 44.45 0)
 			(effects
@@
 			(project "OrangePie"
 				(path "/3103c9de-f1ba-4d51-8bfc-798df1c75e2f/50dedcd5-65c1-4d6e-8d03-473117f8d376"
-					(reference "#PWR083")
+					(reference "#PWR07")
 					(unit 1)
 				)
@@
 		(on_board yes)
 		(dnp no)
-		(property "Reference" "#PWR090"
+		(property "Reference" "#PWR010"
 			(at 138.43 52.07 0)
 			(effects
@@
 			(project "OrangePie"
 				(path "/3103c9de-f1ba-4d51-8bfc-798df1c75e2f/50dedcd5-65c1-4d6e-8d03-473117f8d376"
-					(reference "#PWR090")
+					(reference "#PWR010")
 					(unit 1)
 				)
@@
 		(on_board yes)
 		(dnp no)
-		(property "Reference" "#PWR084"
+		(property "Reference" "#PWR08"
 			(at 138.43 44.45 0)
 			(effects
@@
 			(project "OrangePie"
 				(path "/3103c9de-f1ba-4d51-8bfc-798df1c75e2f/50dedcd5-65c1-4d6e-8d03-473117f8d376"
-					(reference "#PWR084")
+					(reference "#PWR08")
 					(unit 1)
 				)
@@
 		(on_board yes)
 		(dnp no)
-		(property "Reference" "#PWR0112"
+		(property "Reference" "#PWR023"
 			(at 156.21 156.21 0)
 			(effects
@@
 			(project "OrangePie"
 				(path "/3103c9de-f1ba-4d51-8bfc-798df1c75e2f/50dedcd5-65c1-4d6e-8d03-473117f8d376"
-					(reference "#PWR0112")
+					(reference "#PWR023")
 					(unit 1)
 				)
@@
 		(on_board yes)
 		(dnp no)
-		(property "Reference" "J3"
+		(property "Reference" "J1"
 			(at 103.886 15.24 0)
 			(effects
@@
 			(project "OrangePie"
 				(path "/3103c9de-f1ba-4d51-8bfc-798df1c75e2f/50dedcd5-65c1-4d6e-8d03-473117f8d376"
-					(reference "J3")
+					(reference "J1")
 					(unit 1)
 				)
@@
 		(on_board yes)
 		(dnp no)
-		(property "Reference" "#PWR094"
+		(property "Reference" "#PWR012"
 			(at 138.43 57.15 0)
 			(effects
@@
 			(project "OrangePie"
 				(path "/3103c9de-f1ba-4d51-8bfc-798df1c75e2f/50dedcd5-65c1-4d6e-8d03-473117f8d376"
-					(reference "#PWR094")
+					(reference "#PWR012")
 					(unit 1)
 				)
@@
 		(on_board yes)
 		(dnp no)
-		(property "Reference" "#PWR076"
+		(property "Reference" "#PWR02"
 			(at 138.43 21.59 0)
 			(effects
@@
 			(project "OrangePie"
 				(path "/3103c9de-f1ba-4d51-8bfc-798df1c75e2f/50dedcd5-65c1-4d6e-8d03-473117f8d376"
-					(reference "#PWR076")
+					(reference "#PWR02")
 					(unit 1)
 				)
@@
 		(on_board yes)
 		(dnp no)
-		(property "Reference" "#PWR0100"
+		(property "Reference" "#PWR017"
 			(at 71.12 113.03 0)
 			(effects
@@
 			(project "OrangePie"
 				(path "/3103c9de-f1ba-4d51-8bfc-798df1c75e2f/50dedcd5-65c1-4d6e-8d03-473117f8d376"
-					(reference "#PWR0100")
+					(reference "#PWR017")
 					(unit 1)
 				)
@@
 		(on_board yes)
 		(dnp no)
-		(property "Reference" "#PWR075"
+		(property "Reference" "#PWR01"
 			(at 69.85 21.59 0)
 			(effects
@@
 			(project "OrangePie"
 				(path "/3103c9de-f1ba-4d51-8bfc-798df1c75e2f/50dedcd5-65c1-4d6e-8d03-473117f8d376"
-					(reference "#PWR075")
+					(reference "#PWR01")
 					(unit 1)
 				)
@@
 		(on_board yes)
 		(dnp no)
-		(property "Reference" "#PWR082"
+		(property "Reference" "#PWR06"
 			(at 138.43 36.83 0)
 			(effects
@@
 			(project "OrangePie"
 				(path "/3103c9de-f1ba-4d51-8bfc-798df1c75e2f/50dedcd5-65c1-4d6e-8d03-473117f8d376"
-					(reference "#PWR082")
+					(reference "#PWR06")
 					(unit 1)
 				)
@@
 		(on_board yes)
 		(dnp no)
-		(property "Reference" "#PWR0105"
+		(property "Reference" "#PWR021"
 			(at 71.12 135.89 0)
 			(effects
@@
 			(project "OrangePie"
 				(path "/3103c9de-f1ba-4d51-8bfc-798df1c75e2f/50dedcd5-65c1-4d6e-8d03-473117f8d376"
-					(reference "#PWR0105")
+					(reference "#PWR021")
 					(unit 1)
 				)
@@
 		(on_board yes)
 		(dnp no)
-		(property "Reference" "#PWR089"
+		(property "Reference" "#PWR09"
 			(at 69.85 52.07 0)
 			(effects
@@
 			(project "OrangePie"
 				(path "/3103c9de-f1ba-4d51-8bfc-798df1c75e2f/50dedcd5-65c1-4d6e-8d03-473117f8d376"
-					(reference "#PWR089")
+					(reference "#PWR09")
 					(unit 1)
 				)
@@
 		(on_board yes)
 		(dnp no)
-		(property "Reference" "#PWR0108"
+		(property "Reference" "#PWR024"
 			(at 82.55 191.77 0)
 			(effects
@@
 			(project "OrangePie"
 				(path "/3103c9de-f1ba-4d51-8bfc-798df1c75e2f/50dedcd5-65c1-4d6e-8d03-473117f8d376"
-					(reference "#PWR0108")
+					(reference "#PWR024")
 					(unit 1)
 				)
@@
 		(on_board yes)
 		(dnp no)
-		(property "Reference" "#PWR0102"
+		(property "Reference" "#PWR020"
 			(at 71.12 128.27 0)
 			(effects
@@
 			(project "OrangePie"
 				(path "/3103c9de-f1ba-4d51-8bfc-798df1c75e2f/50dedcd5-65c1-4d6e-8d03-473117f8d376"
-					(reference "#PWR0102")
+					(reference "#PWR020")
 					(unit 1)
 				)
@@
 		(on_board yes)
 		(dnp no)
-		(property "Reference" "#PWR096"
+		(property "Reference" "#PWR014"
 			(at 134.62 100.33 0)
 			(effects
@@
 			(project "OrangePie"
 				(path "/3103c9de-f1ba-4d51-8bfc-798df1c75e2f/50dedcd5-65c1-4d6e-8d03-473117f8d376"
-					(reference "#PWR096")
+					(reference "#PWR014")
 					(unit 1)
 				)
@@
 		(on_board yes)
 		(dnp no)
-		(property "Reference" "#PWR093"
+		(property "Reference" "#PWR011"
 			(at 69.85 57.15 0)
 			(effects
@@
 			(project "OrangePie"
 				(path "/3103c9de-f1ba-4d51-8bfc-798df1c75e2f/50dedcd5-65c1-4d6e-8d03-473117f8d376"
-					(reference "#PWR093")
+					(reference "#PWR011")
 					(unit 1)
 				)
@@
 		(on_board yes)
 		(dnp no)
-		(property "Reference" "#PWR097"
+		(property "Reference" "#PWR015"
 			(at 71.12 105.41 0)
 			(effects
@@
 			(project "OrangePie"
 				(path "/3103c9de-f1ba-4d51-8bfc-798df1c75e2f/50dedcd5-65c1-4d6e-8d03-473117f8d376"
-					(reference "#PWR097")
+					(reference "#PWR015")
 					(unit 1)
 				)
@@
 		(on_board yes)
 		(dnp no)
-		(property "Reference" "U13"
+		(property "Reference" "U1"
 			(at 160.02 125.222 0)
 			(effects
@@
 			(project "OrangePie"
 				(path "/3103c9de-f1ba-4d51-8bfc-798df1c75e2f/50dedcd5-65c1-4d6e-8d03-473117f8d376"
-					(reference "U13")
+					(reference "U1")
 					(unit 1)
 				)
@@
 		(on_board yes)
 		(dnp no)
-		(property "Reference" "#PWR0111"
+		(property "Reference" "#PWR019"
 			(at 156.21 128.27 0)
 			(effects
@@
 			(project "OrangePie"
 				(path "/3103c9de-f1ba-4d51-8bfc-798df1c75e2f/50dedcd5-65c1-4d6e-8d03-473117f8d376"
-					(reference "#PWR0111")
+					(reference "#PWR019")
 					(unit 1)
 				)
@@
 		(on_board yes)
 		(dnp no)
-		(property "Reference" "#PWR0101"
+		(property "Reference" "#PWR018"
 			(at 71.12 120.65 0)
 			(effects
@@
 			(project "OrangePie"
 				(path "/3103c9de-f1ba-4d51-8bfc-798df1c75e2f/50dedcd5-65c1-4d6e-8d03-473117f8d376"
-					(reference "#PWR0101")
+					(reference "#PWR018")
 					(unit 1)
 				)
@@
 		(on_board yes)
 		(dnp no)
-		(property "Reference" "#PWR080"
+		(property "Reference" "#PWR04"
 			(at 138.43 29.21 0)
 			(effects
@@
 			(project "OrangePie"
 				(path "/3103c9de-f1ba-4d51-8bfc-798df1c75e2f/50dedcd5-65c1-4d6e-8d03-473117f8d376"
-					(reference "#PWR080")
+					(reference "#PWR04")
 					(unit 1)
 				)
@@
 		(on_board yes)
 		(dnp no)
-		(property "Reference" "#PWR095"
+		(property "Reference" "#PWR013"
 			(at 71.12 100.33 0)
 			(effects
@@
 			(project "OrangePie"
 				(path "/3103c9de-f1ba-4d51-8bfc-798df1c75e2f/50dedcd5-65c1-4d6e-8d03-473117f8d376"
-					(reference "#PWR095")
+					(reference "#PWR013")
 					(unit 1)
 				)
@@
 		(on_board yes)
 		(dnp no)
-		(property "Reference" "#PWR081"
+		(property "Reference" "#PWR05"
 			(at 69.85 36.83 0)
 			(effects
@@
 			(project "OrangePie"
 				(path "/3103c9de-f1ba-4d51-8bfc-798df1c75e2f/50dedcd5-65c1-4d6e-8d03-473117f8d376"
-					(reference "#PWR081")
+					(reference "#PWR05")
 					(unit 1)
 				)

Commit message: Pass ERC
Connections:
- net GPIOR14 renamed USB_IN-
- net GPIOR15 renamed USB_IN+
- net STDBY OUT renamed 5v_STDBY
- net USB1U.D+: no longer names the net of J1.a2
- net USB1U.D-: no longer names the net of J1.c2

Commit message: Prepare board for layout
Connections:
- net CAN1_TR_OUT.+ renamed CAN1_TR_OUT.C+
- net CAN1_TR_OUT.- renamed CAN1_TR_OUT.C-
- net CAN2_TR_OUT.+ renamed CAN2_TR_OUT.C+
- net CAN2_TR_OUT.- renamed CAN2_TR_OUT.C-
- net USB_DEBUG.+ renamed USB_DEBUG.D+
- net USB_DEBUG.- renamed USB_DEBUG.D-
- net USB_IN+ renamed USB_IN.D+
- net USB_IN- renamed USB_IN.D-

Commit message: Do signal layer layout
Parts:
- removed U1: IP4234CZ6,115, Package_TO_SOT_SMD:SC-74-6_1.55x2.9mm_P0.95mm, symbol Power_Protection:IP4234CZ6
- added U14: PESD5V0S2BT, Package_TO_SOT_SMD:SOT-23, symbol PESD5V0S2BT:PESD5V0S2BT
Connections:
- net USB_IN.D+ is gone; now on net USB_DEBUG.D+: J1.c31
- net USB_IN.D- is gone; now on net USB_DEBUG.D-: J1.c30
- net GND: now also U14.3
- net USB_DEBUG.D+: now also U14.1
- net USB_DEBUG.D-: now also U14.2
Other:
- note removed: "USB"

Commit message: Fix schematic
Parts:
- removed U14: PESD5V0S2BT, Package_TO_SOT_SMD:SOT-23, symbol PESD5V0S2BT:PESD5V0S2BT
- added U403: TPD2E2U06DCK, Package_TO_SOT_SMD:SOT-323_SC-70, symbol Power_Protection:TPD2E2U06DCK
Connections:
- net GND: now also U403.3
- net USB_DEBUG.D+: now also U403.1
- net USB_DEBUG.D-: now also U403.2
