File: PCB source/USB HUB.kicad_sch (KiCad schematic)
At the start: 6 parts, among them U3 CH334R, Y1 12MHz

Commit message: Do Cleanup
Parts:
- renumbered C8 to C45, C7 to C46, C16 to C47, C17 to C48, U3 to U10
Other:
- moved on the sheet: C45, C46

Commit message: Prepare board for layout
Connections:
- net USB3.+ renamed USB3.D+
- net USB3.- renamed USB3.D-
- net USB4.+ renamed USB4.D+
- net USB4.- renamed USB4.D-
- net USB_AUDIO.+ renamed USB_CAN.D+
- net USB_AUDIO.- renamed USB_CAN.D-
- net USB_CAN.+ renamed USB_AUDIO.D+
- net USB_CAN.- renamed USB_AUDIO.D-
- net USB_SBC.+ renamed USB_SBC.D+
- net USB_SBC.- renamed USB_SBC.D-

Commit message: Finish layout
Parts:
- removed C48: 100nF, PCM_JLCPCB:C_0402, symbol PCM_JLCPCB-Capacitors:0402,100nF
Other:
- moved on the sheet: C47

Commit message: Fix schematic
Parts:
- C45, C47: Price 0.007USD -> 0.008USD; Stock 9197991 -> 1226257
- C46: Stock 8324208 -> 6453835
