File: PCB source/Power Oring.kicad_sch (KiCad schematic)
At the start: 9 parts, among them Q2 AO3400, Q3 AO3400, Q4 MMBT3904, U7 LM74700, U8 LM74700

Commit message: Do Cleanup
Parts:
- removed Q4: MMBT3904, PCM_JLCPCB:Q_SOT-23, symbol PCM_JLCPCB-Transistors:NPN,MMBT3904
- added Q5: MMBT3904, PCM_JLCPCB:Q_SOT-23, symbol PCM_JLCPCB-Transistors:NPN,MMBT3904
- renumbered C33 to C26, C34 to C27, Q2 to Q1, R18 to R12, R22 to R13, U7 to U4, U8 to U5
Connections:
- net GND: now also Q5.2 (E)
- net ~{STDBY EN}: now also Q5.1 (B)
- net at R13.2, U5.3 (EN): now also Q5.3 (C)
Other:
- note added: "1"
- note added: "2"
- note added: "3"
- note added: "STDBY EN"
- note added: "STDBY ~{EN}"
- note added: "buck off"
- note added: "ok"
- note added: "~{ok}"

Commit message: Pass ERC
Parts:
- removed Q1, Q3: AO3400, Package_TO_SOT_SMD:SOT-23, symbol Simulation_SPICE:NMOS
- added Q1, Q2: AO3400A, Package_TO_SOT_SMD:SOT-23, symbol Transistor_FET:AO3400A
Connections:
- net +5V: now also Q1.3 (D), Q2.3 (D)
- net BUCK_IN: now also Q2.2 (S)
- net STDBY_IN: now also Q1.2 (S)
- net at U5.5 (GATE): now also Q1.1 (G)
- net at U4.5 (GATE): now also Q2.1 (G)
Changed lines of the file:
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@@
+	)
+	(junction
+		(at 243.84 85.09)
+		(diameter 0)
+		(color 0 0 0 0)
 	)
 	(junction
@@
 	(wire
 		(pts
-			(xy 171.45 85.09) (xy 256.54 85.09)
+			(xy 171.45 85.09) (xy 243.84 85.09)
 		)
 		(stroke
@@
 		(pts
 			(xy 85.09 142.24) (xy 111.76 142.24)
+		)
+		(stroke
+			(width 0)
+			(type default)
+		)
+	)
+	(wire
+		(pts
+			(xy 243.84 85.09) (xy 256.54 85.09)
+		)
+		(stroke
+			(width 0)
+			(type default)
+		)
+	)
+	(wire
+		(pts
+			(xy 243.84 81.28) (xy 243.84 85.09)
 		)
 		(stroke
@@
 	)
 	(symbol
+		(lib_id "Transistor_FET:AO3400A")
+		(at 124.46 119.38 270)
+		(mirror x)
+		(unit 1)
+		(exclude_from_sim no)
+		(in_bom yes)
+		(on_board yes)
+		(dnp no)
+		(fields_autoplaced yes)
+		(property "Reference" "Q1"
+			(at 124.46 110.49 90)
+			(effects
+				(font
+					(size 1.27 1.27)
+				)
+			)
+		)
+		(property "Value" "AO3400A"
+			(at 124.46 113.03 90)
+			(effects
+				(font
+					(size 1.27 1.27)
+				)
+			)
+		)
+		(property "Footprint" "Package_TO_SOT_SMD:SOT-23"
+			(at 122.555 114.3 0)
+			(effects
+				(font
+					(size 1.27 1.27)
+					(italic yes)
+				)
+				(justify left)
+				(hide yes)
+			)
+		)
+		(property "Datasheet" "http://www.aosmd.com/pdfs/datasheet/AO3400A.pdf"
+			(at 120.65 114.3 0)
+			(effects
+				(font
+					(size 1.27 1.27)
+				)
+				(justify left)
+				(hide yes)
+			)
+		)
+		(property "Description" "30V Vds, 5.7A Id, N-Channel MOSFET, SOT-23"
+			(at 124.46 119.38 0)
+			(effects
+				(font
+					(size 1.27 1.27)
+				)
+				(hide yes)
+			)
+		)
+		(pin "1"
+		)
+		(pin "2"
+		)
+		(pin "3"
+		)
+		(instances
+			(project "OrangePie"
+				(path "/3103c9de-f1ba-4d51-8bfc-798df1c75e2f/173701d7-f398-4eb9-8378-88f17944d65b"
+					(reference "Q1")
+					(unit 1)
+				)
+			)
+		)
+	)
+	(symbol
 		(lib_id "PCM_JLCPCB-Resistors:0402,10kΩ")
 		(at 85.09 130.81 0)
@@
 	)
 	(symbol
-		(lib_id "Simulation_SPICE:NMOS")
-		(at 124.46 53.34 270)
-		(mirror x)
-		(unit 1)
-		(exclude_from_sim no)
-		(in_bom yes)
-		(on_board yes)
-		(dnp no)
-		(fields_autoplaced yes)
-		(property "Reference" "Q1"
-			(at 124.46 44.45 90)
-			(effects
-				(font
-					(size 1.27 1.27)
-				)
-			)
-		)
-		(property "Value" "AO3400"
-			(at 124.46 46.99 90)
-			(effects
-				(font
-					(size 1.27 1.27)
-				)
-			)
-		)
-		(property "Footprint" "Package_TO_SOT_SMD:SOT-23"
-			(at 127 48.26 0)
-			(effects
-				(font
-					(size 1.27 1.27)
-				)
-				(hide yes)
-			)
-		)
-		(property "Datasheet" "https://ngspice.sourceforge.io/docs/ngspice-html-manual/manual.xhtml#cha_MOSFETs"
-			(at 111.76 53.34 0)
-			(effects
-				(font
-					(size 1.27 1.27)
-				)
-				(hide yes)
-			)
-		)
-		(property "Description" "N-MOSFET transistor, drain/source/gate"
-			(at 121.666 53.34 0)
-			(effects
-				(font
-					(size 1.27 1.27)
-				)
-				(hide yes)
-			)
-		)
-		(property "Sim.Device" "NMOS"
-			(at 107.315 53.34 0)
-			(effects
-				(font
-					(size 1.27 1.27)
-				)
-				(hide yes)
-			)
-		)
-		(property "Sim.Type" "VDMOS"
-			(at 105.41 53.34 0)
-			(effects
-				(font
-					(size 1.27 1.27)
-				)
-				(hide yes)
-			)
-		)
-		(property "Sim.Pins" "1=D 2=G 3=S"
-			(at 109.22 53.34 0)
-			(effects
-				(font
-					(size 1.27 1.27)
-				)
-				(hide yes)
-			)
-		)
-		(pin "2"
-		)
-		(pin "1"
-		)
-		(pin "3"
-		)
-		(instances
-			(project "OrangePie"
-				(path "/3103c9de-f1ba-4d51-8bfc-798df1c75e2f/173701d7-f398-4eb9-8378-88f17944d65b"
-					(reference "Q1")
-					(unit 1)
-				)
-			)
-		)
-	)
-	(symbol
 		(lib_id "Device:C_Small")
 		(at 97.79 130.81 0)
@@
 	)
 	(symbol
-		(lib_id "Simulation_SPICE:NMOS")
-		(at 124.46 119.38 270)
-		(mirror x)
+		(lib_id "power:PWR_FLAG")
+		(at 243.84 81.28 0)
 		(unit 1)
 		(exclude_from_sim no)
@@
 		(dnp no)
 		(fields_autoplaced yes)
-		(property "Reference" "Q3"
-			(at 124.46 110.49 90)
-			(effects
-				(font
-					(size 1.27 1.27)
-				)
-			)
-		)
-		(property "Value" "AO3400"
-			(at 124.46 113.03 90)
+		(property "Reference" "#FLG05"
+			(at 243.84 79.375 0)
+			(effects
+				(font
+					(size 1.27 1.27)
+				)
+				(hide yes)
+			)
+		)
+		(property "Value" "PWR_FLAG"
+			(at 243.84 76.2 0)
+			(effects
+				(font
+					(size 1.27 1.27)
+				)
+			)
+		)
+		(property "Footprint" ""
+			(at 243.84 81.28 0)
+			(effects
+				(font
+					(size 1.27 1.27)
+				)
+				(hide yes)
+			)
+		)
+		(property "Datasheet" "~"
+			(at 243.84 81.28 0)
+			(effects
+				(font
+					(size 1.27 1.27)
+				)
+				(hide yes)
+			)
+		)
+		(property "Description" "Special symbol for telling ERC where power comes from"
+			(at 243.84 81.28 0)
+			(effects
+				(font
+					(size 1.27 1.27)
+				)
+				(hide yes)
+			)
+		)
+		(pin "1"
+		)
+		(instances
+			(project ""
+				(path "/3103c9de-f1ba-4d51-8bfc-798df1c75e2f/173701d7-f398-4eb9-8378-88f17944d65b"
+					(reference "#FLG05")
+					(unit 1)
+				)
+			)
+		)
+	)
+	(symbol
+		(lib_id "Transistor_FET:AO3400A")
+		(at 124.46 53.34 270)
+		(mirror x)
+		(unit 1)
+		(exclude_from_sim no)
+		(in_bom yes)
+		(on_board yes)
+		(dnp no)
+		(fields_autoplaced yes)
+		(property "Reference" "Q2"
+			(at 124.46 44.45 90)
+			(effects
+				(font
+					(size 1.27 1.27)
+				)
+			)
+		)
+		(property "Value" "AO3400A"
+			(at 124.46 46.99 90)
 			(effects
 				(font
@@
 		)
 		(property "Footprint" "Package_TO_SOT_SMD:SOT-23"
-			(at 127 114.3 0)
-			(effects
-				(font
-					(size 1.27 1.27)
-				)
-				(hide yes)
-			)
-		)
-		(property "Datasheet" "https://ngspice.sourceforge.io/docs/ngspice-html-manual/manual.xhtml#cha_MOSFETs"
-			(at 111.76 119.38 0)
-			(effects
-				(font
-					(size 1.27 1.27)
-				)
-				(hide yes)
-			)
-		)
-		(property "Description" "N-MOSFET transistor, drain/source/gate"
-			(at 121.666 119.38 0)
-			(effects
-				(font
-					(size 1.27 1.27)
-				)
-				(hide yes)
-			)
-		)
-		(property "Sim.Device" "NMOS"
-			(at 107.315 119.38 0)
-			(effects
-				(font
-					(size 1.27 1.27)
-				)
-				(hide yes)
-			)
-		)
-		(property "Sim.Type" "VDMOS"
-			(at 105.41 119.38 0)
-			(effects
-				(font
-					(size 1.27 1.27)
-				)
-				(hide yes)
-			)
-		)
-		(property "Sim.Pins" "1=D 2=G 3=S"
-			(at 109.22 119.38 0)
-			(effects
-				(font
-					(size 1.27 1.27)
-				)
-				(hide yes)
-			)
+			(at 122.555 48.26 0)
+			(effects
+				(font
+					(size 1.27 1.27)
+					(italic yes)
+				)
+				(justify left)
+				(hide yes)
+			)
+		)
+		(property "Datasheet" "http://www.aosmd.com/pdfs/datasheet/AO3400A.pdf"
+			(at 120.65 48.26 0)
+			(effects
+				(font
+					(size 1.27 1.27)
+				)
+				(justify left)
+				(hide yes)
+			)
+		)
+		(property "Description" "30V Vds, 5.7A Id, N-Channel MOSFET, SOT-23"
+			(at 124.46 53.34 0)
+			(effects
+				(font
+					(size 1.27 1.27)
+				)
+				(hide yes)
+			)
+		)
+		(pin "1"
 		)
 		(pin "2"
 		)
-		(pin "1"
-		)
 		(pin "3"
 		)
 		(instances
-			(project "OrangePie"
+			(project ""
 				(path "/3103c9de-f1ba-4d51-8bfc-798df1c75e2f/173701d7-f398-4eb9-8378-88f17944d65b"
-					(reference "Q3")
+					(reference "Q2")
 					(unit 1)
 				)

Commit message: Fix schematic
Parts:
- removed Q1, Q2: AO3400A, Package_TO_SOT_SMD:SOT-23, symbol Transistor_FET:AO3400A
- removed Q5: MMBT3904, PCM_JLCPCB:Q_SOT-23, symbol PCM_JLCPCB-Transistors:NPN,MMBT3904
- added Q1, Q2, Q5: AO3400A, PCM_JLCPCB:Q_SOT-23, symbol PCM_JLCPCB-Transistors:NMOS,AO3400A
- R12, R13: Stock 6666349 -> 13746052
Connections:
- net +5V: now also Q1.2 (S), Q2.2 (S)
- net BUCK_IN: now also Q2.3 (D)
- net GND: now also Q5.2 (S)
- net STDBY_IN: now also Q1.3 (D)
- net ~{STDBY EN}: now also Q5.1 (G)
- net at R13.2, U5.3 (EN): now also Q5.3 (D)
- net at U5.5 (GATE): now also Q1.1 (G)
- net at U4.5 (GATE): now also Q2.1 (G)

Commit message: [3] Finish pcb
Connections:
- net +5V: now also Q1.3 (D), Q2.3 (D); no longer Q1.2 (S), Q2.2 (S)
- net BUCK_IN: now also Q2.2 (S); no longer Q2.3 (D)
- net STDBY_IN: now also Q1.2 (S); no longer Q1.3 (D)
Other:
- moved on the sheet: Q1, Q2
Changed lines of the file:
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@@
 	(symbol
 		(lib_id "PCM_JLCPCB-Transistors:NMOS,AO3400A")
-		(at 124.46 53.34 90)
+		(at 124.46 53.34 270)
+		(mirror x)
 		(unit 1)
 		(exclude_from_sim no)
@@
 		(on_board yes)
 		(dnp no)
-		(fields_autoplaced yes)
 		(property "Reference" "Q2"
 			(at 124.46 44.45 90)
@@
 	(symbol
 		(lib_id "PCM_JLCPCB-Transistors:NMOS,AO3400A")
-		(at 124.46 119.38 90)
+		(at 124.46 119.38 270)
+		(mirror x)
 		(unit 1)
 		(exclude_from_sim no)
@@
 		(on_board yes)
 		(dnp no)
-		(fields_autoplaced yes)
 		(property "Reference" "Q1"
 			(at 124.46 110.49 90)
