File: PCB source/Can Transiver.kicad_sch (KiCad schematic)
At the start: 4 parts, among them U4 TJA1044GTK_3Z

Commit message: Do Cleanup
Parts:
- removed C18, C19: 100nF, Capacitor_SMD:C_0402_1005Metric, symbol Device:C_Small
- removed R8: 10k, Resistor_SMD:R_0402_1005Metric, symbol Device:R_Small
- added C28, C29: 100nF, PCM_JLCPCB:C_0402, symbol PCM_JLCPCB-Capacitors:0402,100nF,(2)
- added R14: 10kΩ, PCM_JLCPCB:R_0402, symbol PCM_JLCPCB-Resistors:0402,10kΩ
- renumbered U4 to U6
Connections:
- net +3V3: now also C29.1
- net +5V: now also C28.2
- net GND: now also C28.1, C29.2, R14.2
- net at U6.8 (STB): now also R14.1

Commit message: Prepare board for layout
Connections:
- net CAN_TR_OUT.+ renamed CAN_TR_OUT.C+
- net CAN_TR_OUT.- renamed CAN_TR_OUT.C-
Changed lines of the file:
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@@
 	)
 	(bus_alias "CAN"
-		(members "+" "-")
+		(members "C+" "C-")
 	)
 	(junction
@@
 		)
 	)
-	(label "CAN_TR_OUT.+"
+	(label "CAN_TR_OUT.C+"
 		(at 153.67 100.33 0)
 		(fields_autoplaced yes)
@@
 		)
 	)
-	(label "CAN_TR_OUT.-"
+	(label "CAN_TR_OUT.C-"
 		(at 153.67 102.87 0)
 		(fields_autoplaced yes)

Commit message: Add 22R resistors to USB
Parts:
- removed R14: 10kΩ, PCM_JLCPCB:R_0402, symbol PCM_JLCPCB-Resistors:0402,10kΩ
- added R34: 0Ω, PCM_JLCPCB:R_0402, symbol PCM_JLCPCB-Resistors:0402,0Ω
Connections:
- net GND: now also R34.2
- net at U6.8 (STB): now also R34.1

Commit message: Fix schematic
Parts:
- C28, C29: Stock 5358037 -> 5436546
- R34: Stock 5514860 -> 6249348
Connections:
- net +3V3 renamed CAN_3V3
Changed lines of the file:
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@@
 (kicad_sch
-	(version 20231120)
+	(version 20250114)
 	(generator "eeschema")
-	(generator_version "8.0")
+	(generator_version "9.0")
 	(paper "A4")
 	(title_block
@@
 	)
 	(junction
+		(at 124.46 90.17)
+		(diameter 0)
+		(color 0 0 0 0)
+	)
+	(junction
 		(at 149.86 91.44)
 		(diameter 0)
 		(color 0 0 0 0)
 	)
-	(junction
-		(at 124.46 90.17)
-		(diameter 0)
-		(color 0 0 0 0)
-	)
 	(bus_entry
 		(at 171.45 97.79)
@@
 	(wire
 		(pts
+			(xy 149.86 71.12) (xy 156.21 71.12)
+		)
+		(stroke
+			(width 0)
+			(type default)
+		)
+	)
+	(wire
+		(pts
 			(xy 111.76 92.71) (xy 111.76 90.17)
 		)
@@
 	(wire
 		(pts
-			(xy 149.86 88.9) (xy 149.86 91.44)
+			(xy 149.86 91.44) (xy 149.86 71.12)
 		)
 		(stroke
@@
 	(label "CAN_TR.TXD"
 		(at 110.49 100.33 0)
-		(fields_autoplaced yes)
 		(effects
 			(font
@@
 	(label "CAN_TR_OUT.C+"
 		(at 153.67 100.33 0)
-		(fields_autoplaced yes)
 		(effects
 			(font
@@
 	(label "CAN_TR.RXD"
 		(at 110.49 102.87 0)
-		(fields_autoplaced yes)
 		(effects
 			(font
@@
 	(label "CAN_TR_OUT.C-"
 		(at 153.67 102.87 0)
-		(fields_autoplaced yes)
 		(effects
 			(font
@@
 		(shape input)
 		(at 176.53 93.98 0)
-		(fields_autoplaced yes)
 		(effects
 			(font
@@
 		(shape input)
 		(at 96.52 93.98 180)
-		(fields_autoplaced yes)
 		(effects
 			(font
@@
 			)
 			(justify right)
+		)
+	)
+	(hierarchical_label "CAN_3V3"
+		(shape input)
+		(at 156.21 71.12 0)
+		(effects
+			(font
+				(size 1.27 1.27)
+			)
+			(justify left)
 		)
 	)
@@
 			)
 		)
-		(property "Stock" "5358037"
+		(property "Stock" "5436546"
 			(at 116.84 90.17 0)
 			(effects
@@
 				(path "/3103c9de-f1ba-4d51-8bfc-798df1c75e2f/90c85cbd-0f83-4bab-9a58-f576d03aa82a"
 					(reference "C30")
-					(unit 1)
-				)
-			)
-		)
-	)
-	(symbol
-		(lib_id "power:+5V")
-		(at 149.86 88.9 0)
-		(unit 1)
-		(exclude_from_sim no)
-		(in_bom yes)
-		(on_board yes)
-		(dnp no)
-		(property "Reference" "#PWR063"
-			(at 149.86 92.71 0)
-			(effects
-				(font
-					(size 1.27 1.27)
-				)
-				(hide yes)
-			)
-		)
-		(property "Value" "+3V3"
-			(at 149.86 85.09 0)
-			(effects
-				(font
-					(size 1.27 1.27)
-				)
-			)
-		)
-		(property "Footprint" ""
-			(at 149.86 88.9 0)
-			(effects
-				(font
-					(size 1.27 1.27)
-				)
-				(hide yes)
-			)
-		)
-		(property "Datasheet" ""
-			(at 149.86 88.9 0)
-			(effects
-				(font
-					(size 1.27 1.27)
-				)
-				(hide yes)
-			)
-		)
-		(property "Description" "Power symbol creates a global label with name \"+5V\""
-			(at 149.86 88.9 0)
-			(effects
-				(font
-					(size 1.27 1.27)
-				)
-				(hide yes)
-			)
-		)
-		(pin "1"
-		)
-		(instances
-			(project "OrangePie"
-				(path "/3103c9de-f1ba-4d51-8bfc-798df1c75e2f/4ef8679b-7d0c-4776-8ce3-817c4ec1763f"
-					(reference "#PWR063")
-					(unit 1)
-				)
-				(path "/3103c9de-f1ba-4d51-8bfc-798df1c75e2f/90c85cbd-0f83-4bab-9a58-f576d03aa82a"
-					(reference "#PWR069")
 					(unit 1)
 				)
@@
 			)
 		)
-		(property "Stock" "5514860"
+		(property "Stock" "6249348"
 			(at 149.86 113.03 0)
 			(effects
@@
 			)
 		)
-		(property "Stock" "5358037"
+		(property "Stock" "5436546"
 			(at 157.48 91.44 0)
 			(effects

Commit message: Fix can power delivery , fixed placment of the mosfets, CAN power  pull down to avoid DFU boot, added new porgraming connector
Connections:
- net +5V renamed CAN_5V
Changed lines of the file:
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@@
+	(wire
+		(pts
+			(xy 127 72.39) (xy 124.46 72.39)
+		)
+		(stroke
+			(width 0)
+			(type default)
+		)
+	)
 	(wire
 		(pts
@@
 	(wire
 		(pts
-			(xy 149.86 71.12) (xy 156.21 71.12)
+			(xy 149.86 72.39) (xy 152.4 72.39)
 		)
 		(stroke
@@
 	(wire
 		(pts
+			(xy 124.46 72.39) (xy 124.46 90.17)
+		)
+		(stroke
+			(width 0)
+			(type default)
+		)
+	)
+	(wire
+		(pts
 			(xy 147.32 102.87) (xy 168.91 102.87)
 		)
@@
 	(wire
 		(pts
-			(xy 149.86 91.44) (xy 149.86 71.12)
+			(xy 149.86 91.44) (xy 149.86 72.39)
 		)
 		(stroke
@@
 		(pts
 			(xy 149.86 109.22) (xy 149.86 107.95)
-		)
-		(stroke
-			(width 0)
-			(type default)
-		)
-	)
-	(wire
-		(pts
-			(xy 124.46 88.9) (xy 124.46 90.17)
 		)
 		(stroke
@@
 		)
 	)
+	(hierarchical_label "CAN_5V"
+		(shape input)
+		(at 127 72.39 0)
+		(effects
+			(font
+				(size 1.27 1.27)
+			)
+			(justify left)
+		)
+	)
 	(hierarchical_label "CAN_3V3"
 		(shape input)
-		(at 156.21 71.12 0)
+		(at 152.4 72.39 0)
 		(effects
 			(font
@@
 		)
 	)
-	(symbol
-		(lib_id "power:+5V")
-		(at 124.46 88.9 0)
-		(unit 1)
-		(exclude_from_sim no)
-		(in_bom yes)
-		(on_board yes)
-		(dnp no)
-		(property "Reference" "#PWR062"
-			(at 124.46 92.71 0)
-			(effects
-				(font
-					(size 1.27 1.27)
-				)
-				(hide yes)
-			)
-		)
-		(property "Value" "+5V"
-			(at 124.46 85.09 0)
-			(effects
-				(font
-					(size 1.27 1.27)
-				)
-			)
-		)
-		(property "Footprint" ""
-			(at 124.46 88.9 0)
-			(effects
-				(font
-					(size 1.27 1.27)
-				)
-				(hide yes)
-			)
-		)
-		(property "Datasheet" ""
-			(at 124.46 88.9 0)
-			(effects
-				(font
-					(size 1.27 1.27)
-				)
-				(hide yes)
-			)
-		)
-		(property "Description" "Power symbol creates a global label with name \"+5V\""
-			(at 124.46 88.9 0)
-			(effects
-				(font
-					(size 1.27 1.27)
-				)
-				(hide yes)
-			)
-		)
-		(pin "1"
-		)
-		(instances
-			(project "OrangePie"
-				(path "/3103c9de-f1ba-4d51-8bfc-798df1c75e2f/4ef8679b-7d0c-4776-8ce3-817c4ec1763f"
-					(reference "#PWR062")
-					(unit 1)
-				)
-				(path "/3103c9de-f1ba-4d51-8bfc-798df1c75e2f/90c85cbd-0f83-4bab-9a58-f576d03aa82a"
-					(reference "#PWR068")
-					(unit 1)
-				)
-			)
-		)
-	)
